File: hellen121vag.kicad_pcb (KiCad board)
At the start: 4 copper layers, 164 x 118 mm, 129 parts, among them J1 USB_B_Mini, J10 AudioJack_THR, J2 Conn_01x01, J3 Conn_01x01, J4 Conn_01x01, J5 Conn_01x01, J6 Conn_01x01, J7 Conn_01x08, J8 Conn_01x06, M1 Module-can-0.1, M10 Module-can-0.1, M11 Module-vr-discrete-0.1, M2 Module-power5-0.2, M3 Module-mcu-0.7, M4 Module-input-0.1, M5 Module-knock-0.1, M6 Module-output-0.3, M7 Module-ign8-0.2, M8 Module-power12-0.2, M9 Module-wbo-0.3, P1 368255-2, P10 Pad, P11 Pad, P12 Pad, P13 Pad, P14 Pad, P15 Pad, P16 Pad, P17 Pad, P2 Pad, P20 Pad, P28 Pad, P3 Pad, P4 Pad, P40 Pad, P41 Pad, P43 Pad, P44 Pad, P45 Pad, P46 Pad, P48 Pad, P49 Pad, P5 Pad, P56 Pad, P6 Pad, P61 Pad, P63 Pad, P64 Pad, P66 Pad, P67 Pad, P68 Pad, P69 Pad, P7 Pad, P74 Pad, P8 Pad, P80 Pad, P9 Pad, U1 L6205PD, U2 LPS25HB, U3 MCP6002-xSN, U4 TLS115_SOIC, U5 TLS115_SON

Commit message: wew
Parts:
- moved U4 36.1 mm to (57.7, 62.6)
- moved C18 34.2 mm to (60.5, 69.5)
- moved C19 34.2 mm to (60.5, 67.6)
- moved U5 34.2 mm to (56.2, 68.9)

Commit message: weu
Parts:
- moved C18 5.70 mm to (56.0, 73.0)
- moved U4 2.16 mm to (55.7, 61.8)
- moved U5 1.54 mm to (55.4, 67.6)
Changed lines of the file:
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@@
 	(footprint "Package_SON:HVSON-8-1EP_3x3mm_P0.65mm_EP1.6x2.4mm"
 		(layer "F.Cu")
-		(at 56.177499 68.935014)
+		(at 55.4 67.6)
 		(descr "HVSON, 8 Pin (https://www.nxp.com/docs/en/data-sheet/TJA1051.pdf#page=16), generated with kicad-footprint-generator ipc_noLead_generator.py")
 		(tags "HVSON NoLead")
@@
 	(footprint "hellen-one-common:C0603"
 		(layer "F.Cu")
-		(at 60.5375 69.55)
+		(at 56 73)
 		(property "Reference" "C18"
 			(at -0.708119 -0.74013 0)
@@
 	(footprint "kicad6-libraries:PG-DSO-8-43_VIA"
 		(layer "F.Cu")
-		(at 57.655 62.595)
+		(at 55.6625 61.75)
 		(descr "Infineon_PG-DSO-8-43")
 		(tags "DSO DSO-8 SOIC SOIC-8")

Commit message: weu
Parts:
- removed C18: 1u, hellen-one-common:C0603
Routing:
- removed copper zone on In1.Cu, net GND

Commit message: weu
Parts:
- removed C19: 1u, hellen-one-common:C0603
- removed U4: TLS115_SOIC, kicad6-libraries:PG-DSO-8-43_VIA
- removed U5: TLS115_SON, Package_SON:HVSON-8-1EP_3x3mm_P0.65mm_EP1.6x2.4mm

Commit message: weu
Parts:
- removed C15, C6: 100n, hellen-one-common:C0603
- removed M1, M10: Module-can-0.1, hellen-one-can-0.1:can
- removed M2: Module-power5-0.2, hellen-one-power5-0.2:power5
- removed M4: Module-input-0.1, hellen-one-input-0.1:input
- removed R18, R19: 4.7k, hellen-one-common:R0603
- removed R6, R7: 2.7k, hellen-one-common:R0603
- removed S1, S2: Button_SPST, hellen-one-common:SMD-2_2.9x3.9x1.7
- removed U2: LPS25HB, Package_LGA:ST_HLGA-10_2.5x2.5mm_P0.6mm_LayoutBorder3x2y
- M11: value Module-vr-discrete-0.1 -> Module-vr-discrete-0.4; footprint hellen-one-vr-discrete-0.1:vr-discrete -> hellen-one-vr-discrete-0.4:vr-discrete
- M3: value Module-mcu-0.7 -> mega-mcu144-0.1; footprint hellen-one-mcu-0.7:mcu -> hellen-one-mega-mcu144-0.1:mega-mcu144
- M5: value Module-knock-0.1 -> Module-knock-0.2; footprint hellen-one-knock-0.1:knock -> hellen-one-knock-0.2:knock
- M8: value Module-power12-0.2 -> Module-power_12and5V-0.1; footprint hellen-one-power12-0.2:power12 -> hellen-one-power_12and5V-0.1:power_12and5V
- M9: value Module-wbo-0.3 -> Module-wbo-0.5; footprint hellen-one-wbo-0.3:wbo -> hellen-one-wbo-0.5:wbo
- moved M5 19.5 mm to (68.5, 78.7), turned to 0 degrees
Connections:
- M3 pad E14: /+ETB -> /VVT2_B1
- M3 pad E15: /-ETB -> /VVT2_B2
- M3 pad E16: /VVT2_B2 -> /-ETB
- M3 pad E17: /VVT2_B1 -> /+ETB
- M3 pad E18: /THRESHOLD_VR -> /INJ2
- M3 pad E19: /FUEL_CONSUM -> /INJ1
- M3 pad E21: /VVT1_2 -> /IDLE
- M3 pad E23: /IDLE -> /VVT1_2
- M3 pad E25: /INJ1 -> /FUEL_CONSUM
- M3 pad E26: /INJ2 -> /THRESHOLD_VR
- M3 pad N1: /CAN_VIO -> unconnected-(M3-USBID-PadN1)
- M3 pad N10: /SPI3_MISO -> /SPI3_CS
- M3 pad N11: /SPI3_MOSI -> /SPI3_SCK
- M3 pad N12: unconnected-(M3-PadN12) -> /SPI3_MISO
- M3 pad N13: unconnected-(M3-PadN13) -> /SPI3_MOSI
- M3 pad N16: +3V3 -> unconnected-(M3-IO1-PadN16)
- M3 pad N17: /VBAT -> /TX2
- M3 pad N18: Net-(R19-Pad2) -> /RX2
- M3 pad N19: Net-(R18-Pad2) -> unconnected-(M3-IO2-PadN19)
- M3 pad N2: /CAN_RX -> /USBM
- M3 pad N24: /NRESET -> /RX1
- M3 pad N25: unconnected-(M3-PadN25) -> /TX1
- M3 pad N26: unconnected-(M3-PadN26) -> /VIGN
- M3 pad N27: unconnected-(M3-PadN27) -> /VBAT
- M3 pad N28: /BOOT0 -> +5V
- M3 pad N29: /VBUS -> +3V3
- M3 pad N3: /CAN_TX -> /USBP
- M3 pad N4: /TX1 -> /VBUS
- M3 pad N5: /RX1 -> unconnected-(M3-BOOT0-PadN5)
- M3 pad N6: /TX2 -> unconnected-(M3-SWO-PadN6)
- M3 pad N7: /RX2 -> unconnected-(M3-SWDIO-PadN7)
- M3 pad N8: /SPI3_CS -> unconnected-(M3-SWCLK-PadN8)
- M3 pad N9: /SPI3_SCK -> unconnected-(M3-nReset-PadN9)
- M3 pad S1: +5V -> /IN_D4
- M3 pad S10: unconnected-(M3-PadS10) -> /IN_CAM2
- M3 pad S11: unconnected-(M3-PadS11) -> /IN_A3
- M3 pad S12: /KNOCK1 -> /IN_PPS2
- M3 pad S13: /CRANK -> /IN_TPS2
- M3 pad S14: /VSS -> /IN_RES2
- M3 pad S15: /CAM1 -> /IN_A1
- M3 pad S16: /AFR -> /IN_AFR
- M3 pad S17: /TPS1 -> /IN_RES1
- M3 pad S18: /CLT -> /IN_A4
- M3 pad S19: /IAT -> /IN_A2
- M3 pad S2: GND -> /IN_D3
- M3 pad S20: /MAF -> /IN_MAP2
- M3 pad S21: /MAP2 -> /IN_MAF
- M3 pad S22: /A2 -> /IN_CRANK
- M3 pad S23: /A4 -> /IN_KNOCK1
- M3 pad S24: /TPS2 -> /IN_CAM1
- M3 pad S25: /PPS2 -> /IN_VSS
- M3 pad S26: /A3 -> /IN_IAT
- M3 pad S27: /CAM2 -> unconnected-(M3-IN_AT1-PadS27)
- M3 pad S28: /RES1 -> /IN_CLT
- M3 pad S29: /PPS1 -> unconnected-(M3-IN_AT2-PadS29)
- M3 pad S3: /D1 -> /IN_D2
- M3 pad S30: /A1 -> /IN_TPS1
- M3 pad S31: /RES2 -> /IN_PPS1
- M3 pad S32: GNDA -> unconnected-(M3-IN_TPS2-PadS32)
- M3 pad S33: +5VA -> unconnected-(M3-IN_PPS2-PadS33)
- M3 pad S4: /D2 -> /IN_D1
- M3 pad S5: /D3 -> unconnected-(M3-VREF2-PadS5)
- M3 pad S6: /D4 -> unconnected-(M3-IN_SENS4-PadS6)
- M3 pad S7: /VIGN -> unconnected-(M3-IN_SENS3-PadS7)
- M3 pad S8: /VR_ANALOG -> unconnected-(M3-IN_SENS2-PadS8)
- M3 pad S9: unconnected-(M3-PadS9) -> /VR_ANALOG
- M3 pad W1: /IGN1 -> /IGN8
- M3 pad W10: /IGN_V33 -> /CAN-
- M3 pad W2: /IGN2 -> /IGN7
- M3 pad W3: /IGN3 -> /IGN6
- M3 pad W4: /IGN4 -> /IGN5
- M3 pad W5: /IGN5 -> /IGN4
- M3 pad W6: /IGN6 -> /IGN3
- M3 pad W7: /IGN7 -> /IGN2
- M3 pad W8: /IGN8 -> /IGN1
- M3 pad W9: /IGN_V5 -> /CAN+
- M8 pad E1: +5V -> /VBAT
- M8 pad E2: +12V_RAW -> +12V
- M8 pad V1: +12V -> /V12_PERM
- M8 pad V2: /VBAT -> /IN_VIGN
- M8 pad V3: /IN_VIGN -> +12V_RAW
- M8 pad V4: /V12_PERM -> +5VP
- M9 pad W2: Net-(M10-PadV2) -> unconnected-(M9-CAN_VIO-PadW2)
- M9 pad W3: Net-(M10-PadV6) -> /CAN-
- M9 pad W4: Net-(M10-PadV5) -> /CAN+
Routing:
- net +5V: track 359.2 -> 301.1 mm, vias 4 -> 3
- net /IN_D1: track 37.2 -> 95.3 mm, vias 1 -> 2
- net unconnected-(M3-SWDIO-PadN7): track 0.00 -> 46.9 mm, vias 0 -> 2
- net GND: track 109.8 -> 155.5 mm, vias 125 -> 126
- net Net-(R18-Pad2): track 34.1 -> 0.00 mm, vias 1 -> 0
- net unconnected-(M3-SWCLK-PadN8): track 0.00 -> 33.5 mm, vias 0 -> 1
- net Net-(R19-Pad2): track 33.5 -> 0.00 mm, vias 1 -> 0
- net /USBP: track 7.46 -> 33.0 mm, vias 0 -> 1
- net /BOOT0: track 25.5 -> 0.00 mm, vias 1 -> 0
- net /CAN_RX: track 13.0 -> 0.00 mm
- net /NRESET: track 12.8 -> 0.00 mm, vias 1 -> 0
- net /CAN_TX: track 10.2 -> 0.00 mm
- net +5VA: track 16.1 -> 5.97 mm, vias 1 -> 0
- net unconnected-(M9-CAN_VIO-PadW2): track 0.00 -> 8.48 mm
- net Net-(M10-PadV2): track 8.48 -> 0.00 mm
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
Commit message: weu
Parts:
- removed C1, C2: 100n, hellen-one-common:C0603
- removed C10, C11, C12, C13, C14, C7, C8, C9: 10u, Capacitor_SMD:C_0805_2012Metric
- removed C3: 220n, hellen-one-common:C0603
- removed C4: 10n, hellen-one-common:C0603
- removed C5: 5.6n, hellen-one-common:C0603
- removed D1, D2: 1N4148WS, hellen-one-common:SOD-323
- removed R1: 100, hellen-one-common:R0603
- removed R22: 10k, hellen-one-common:R0603
- removed R5: 100k, hellen-one-common:R0603
- removed U1: L6205PD, hellen-one-common:SO20POWER
- added M1: Module-motor-driver-0.1, hellen-one-motor-driver-0.1:motor-driver, F.Cu at (157.6, 17.6)
Routing:
- net +12V_RAW: track 567.8 -> 450.9 mm, vias 18 -> 10
- net /+ETB_OUT: track 0.00 -> 65.4 mm, vias 0 -> 4
- net /-ETB_OUT: track 0.00 -> 51.5 mm, vias 0 -> 4
- net (no net): track 0.00 -> 41.0 mm, vias 0 -> 2
- net Net-(D2-K): track 32.2 -> 0.00 mm, vias 2 -> 0
- net Net-(U1-VCP): track 4.59 -> 0.00 mm
- net Net-(D1-K): track 2.80 -> 0.00 mm
- net Net-(C4-Pad2): track 1.42 -> 0.00 mm

Commit message: weu
Parts:
- moved M1 2.94 mm to (155.9, 20.0)
Changed lines of the file:
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@@
 	(footprint "hellen-one-motor-driver-0.1:motor-driver"
 		(layer "F.Cu")
-		(at 157.6 17.6)
+		(at 155.9 20)
 		(property "Reference" "M1"
 			(at 2.45 -9.8 0)
@@
 			(polygon
 				(pts
-					(xy 171.3 17.5) (xy 157.7 17.5) (xy 157.7 7.7) (xy 171.3 7.7)
+					(xy 169.6 19.9) (xy 156 19.9) (xy 156 10.1) (xy 169.6 10.1)
 				)
 			)

Commit message: fg
Parts:
- removed BT1: BATTERY_CR2032, Battery:BatteryHolder_Keystone_1060_1x2032
- removed C16: 100n, hellen-one-common:C0603
- removed C17: 10u, hellen-one-common:C0603
- removed D10, D11, D12, D13, D14: B5819W, Diode_SMD:D_SOD-123
- removed D7, D8: LED-GREEN-0805, hellen-one-common:LED-0805
- removed D9: 1N4148WS, hellen-one-common:SOD-323
- removed G1, G2, G3, G5: PROTO_AREA, hellen-one-common:PROTO_AREA
- removed G4: DISCLAIMER, rusefi_lib:Off_Road_Disclaimer
- removed G6: LOGO, hellen-one-common:LOGO
- removed G7: LOGO, rusefi_lib:LOGO
- removed J10: AudioJack_THR, hellen-one-common:Jack_3.5mm_PJ-3250-5A
- removed J3, J4, J5, J6: Conn_01x01, TestPoint:TestPoint_Pad_D2.0mm
- removed J7: Conn_01x08, Connector_PinHeader_2.54mm:PinHeader_1x08_P2.54mm_Vertical
- removed J8: Conn_01x06, Connector_PinHeader_2.54mm:PinHeader_1x06_P2.54mm_Vertical
- removed M11: Module-vr-discrete-0.4, hellen-one-vr-discrete-0.4:vr-discrete
- removed M9: Module-wbo-0.5, hellen-one-wbo-0.5:wbo
- removed P10, P11, P12, P13, P14, P15, P16, P17, P20, P28, P3, P4, P40, P41, P43, P44, P45, P46, P48, P49, P5, P56, P6, P61, P63, P64, P66, P67, P68, P69, P7, P74, P8, P80, P9: Pad, hellen-one-common:PAD-TH
- added C1: 10n, hellen-one-common:C0603, F.Cu at (84.4, 71.3)
- added C2: 100n, hellen-one-common:C0603, F.Cu at (84.4, 73.3)
- added C3: 10n, hellen-one-common:C0603, F.Cu at (84.4, 75.2)
- added C4: 100n, hellen-one-common:C0603, F.Cu at (84.4, 77.2)
- added C5: 1u, hellen-one-common:C0603, F.Cu at (84.4, 79.1)
- added D1: B5819W, hellen-one-common:SOD-123, F.Cu at (137.7, 51.7)
- added D2: B5819W, hellen-one-common:SOD-123, F.Cu at (137.7, 54.8)
- added F3: 12H1500D, hellen-one-common:PAD-1206-PAD, F.Cu at (111.4, 66.4)
- added F4: 50mA, Fuse:Fuse_0603_1608Metric, F.Cu at (159.7, 31.7)
- added F5: 50mA, Fuse:Fuse_0603_1608Metric, F.Cu at (159.7, 34.2)
- added F6: 50mA, Fuse:Fuse_0603_1608Metric, F.Cu at (159.7, 36.7)
- added F7: 50mA, Fuse:Fuse_0603_1608Metric, F.Cu at (159.7, 39.2)
- added F8: 50mA, Fuse:Fuse_0603_1608Metric, F.Cu at (159.7, 41.8)
- added F9: 50mA, Fuse:Fuse_0603_1608Metric, F.Cu at (159.7, 44.3)
- added L1: 470R@100MHz, Inductor_SMD:L_0603_1608Metric, F.Cu at (88.1, 78.2)
- added L2: 470R@100MHz, Inductor_SMD:L_0603_1608Metric, F.Cu at (88.1, 80.7)
- added M2: Module-knock-0.2, hellen-one-knock-0.2:knock, F.Cu at (133.7, 60.9)
- added M4: Module-vr-max9924-0.1, hellen-one-vr-max9924-0.1:vr-max9924, F.Cu at (118.7, 27.4)
- added Q1: AO3400A, Package_TO_SOT_SMD:SOT-23, F.Cu at (136.8, 8.41)
- added Q2: ISL9V3040D3ST, Package_TO_SOT_SMD:TO-252-2, F.Cu at (152.4, 10.2)
- added Q3: ISL9V3040D3ST, Package_TO_SOT_SMD:TO-252-2, F.Cu at (152.4, 18.4)
- added Q4: ISL9V3040D3ST, Package_TO_SOT_SMD:TO-252-2, F.Cu at (152.4, 26.6)
- added Q5: ISL9V3040D3ST, Package_TO_SOT_SMD:TO-252-2, F.Cu at (152.4, 34.8)
- added Q6: ISL9V3040D3ST, Package_TO_SOT_SMD:TO-252-2, F.Cu at (152.4, 43.0)
- added Q7: ISL9V3040D3ST, Package_TO_SOT_SMD:TO-252-2, F.Cu at (152.4, 51.2)
- added R1: 4.7k, hellen-one-common:R0603, F.Cu at (137.8, 29.1)
- added R14: 1k, hellen-one-common:R0603, F.Cu at (137.8, 38.8)
- added R15: 4.7k, hellen-one-common:R0603, F.Cu at (111.9, 77.9)
- added R18: 4.7k, hellen-one-common:R0603, F.Cu at (111.9, 79.9)
- added R19: 22, hellen-one-common:R0603, F.Cu at (163.3, 31.4)
- added R22: 0, Resistor_SMD:R_2512_6332Metric, F.Cu at (162.0, 8.45)
- added R24: 0, Resistor_SMD:R_2512_6332Metric, F.Cu at (162.0, 13.3)
- added R25: 22, hellen-one-common:R0603, F.Cu at (163.3, 33.4)
- added R26: 22, hellen-one-common:R0603, F.Cu at (163.3, 35.3)
- added R27: 22, hellen-one-common:R0603, F.Cu at (163.3, 37.3)
- added R28: 0, Resistor_SMD:R_2512_6332Metric, F.Cu at (162.0, 18.2)
- added R29: 0, Resistor_SMD:R_2512_6332Metric, F.Cu at (162.0, 23.1)
- added R30: 0, Resistor_SMD:R_2512_6332Metric, F.Cu at (162.0, 28.0)
- added R31: 4.7k, hellen-one-common:R0603, F.Cu at (155.6, 58.2)
- added R32: 4.7k, hellen-one-common:R0603, F.Cu at (155.6, 60.1)
- added R33: 4.7k, hellen-one-common:R0603, F.Cu at (155.6, 62.1)
- added R34: 4.7k, hellen-one-common:R0603, F.Cu at (155.6, 64.0)
- added R35: 4.7k, hellen-one-common:R0603, F.Cu at (155.6, 65.9)
- added R36: 4.7k, hellen-one-common:R0603, F.Cu at (155.6, 67.9)
- added R37: 4.7k, hellen-one-common:R0603, F.Cu at (158.9, 58.2)
- added R38: 4.7k, hellen-one-common:R0603, F.Cu at (158.9, 60.1)
- added R39: 4.7k, hellen-one-common:R0603, F.Cu at (158.9, 62.1)
- added R40: 4.7k, hellen-one-common:R0603, F.Cu at (158.9, 64.0)
- added R41: 4.7k, hellen-one-common:R0603, F.Cu at (158.9, 65.9)
- added R42: 4.7k, hellen-one-common:R0603, F.Cu at (158.9, 67.9)
- added R43: 4.7k, hellen-one-common:R0603, F.Cu at (162.2, 58.2)
- added R44: 4.7k, hellen-one-common:R0603, F.Cu at (162.2, 60.1)
- added R45: 4.7k, hellen-one-common:R0603, F.Cu at (162.2, 62.1)
- added R46: 4.7k, hellen-one-common:R0603, F.Cu at (162.2, 64.0)
- added R47: 4.7k, hellen-one-common:R0603, F.Cu at (98.2, 71.3)
- added R48: 4.7k, hellen-one-common:R0603, F.Cu at (98.2, 73.3)
- added R49: 4.7k, hellen-one-common:R0603, F.Cu at (98.2, 75.2)
- added R5: 0, hellen-one-common:R0603, F.Cu at (137.8, 34.9)
- added R50: 4.7k, hellen-one-common:R0603, F.Cu at (98.2, 77.2)
- added R6: 0, hellen-one-common:R0603, F.Cu at (137.8, 36.9)
- added R7: DNP, hellen-one-common:R0805, F.Cu at (138.1, 41.0)
- added U1: BTS6143D, Package_TO_SOT_SMD:TO-252-4, F.Cu at (102.2, 62.6)
- added U2: MAX31855KASA, Package_SO:SOIC-8_3.9x4.9mm_P1.27mm, F.Cu at (90.3, 73.7)
- added U4: VNLD5160TR-E, Package_SO:SOIC-8_3.9x4.9mm_P1.27mm, F.Cu at (149.7, 60.5)
- added U5: VNLD5160TR-E, Package_SO:SOIC-8_3.9x4.9mm_P1.27mm, F.Cu at (149.7, 67.1)
- added U6: VNLD5160TR-E, Package_SO:SOIC-8_3.9x4.9mm_P1.27mm, F.Cu at (149.7, 73.7)
- added U7: VNLD5160TR-E, Package_SO:SOIC-8_3.9x4.9mm_P1.27mm, F.Cu at (149.7, 80.3)
- added U8: VNLD5160TR-E, Package_SO:SOIC-8_3.9x4.9mm_P1.27mm, F.Cu at (104.1, 73.7)
- D3: value 1N4148WS -> B5819W; footprint hellen-one-common:SOD-323 -> hellen-one-common:SOD-123
- D4: value LED-GREEN-0805 -> B5819W; footprint hellen-one-common:LED-0805 -> hellen-one-common:SOD-123
- D5: value 1N4148WS -> SS34; footprint hellen-one-common:SOD-323 -> Diode_SMD:D_SMA
- D6: value LED-GREEN-0805 -> NUP2105L; footprint hellen-one-common:LED-0805 -> Package_TO_SOT_SMD:SOT-23
- F1, F2: value Fuse-Pad-Pad -> 12H1500D
- J1: value USB_B_Mini -> Conn_01x05_Male; footprint hellen-one-common:USB-MINI-B-VERTICAL -> Connector_Molex:Molex_SPOX_5267-05A_1x05_P2.50mm_Vertical
- J2: value Conn_01x01 -> USB_B_Mini; footprint TestPoint:TestPoint_Pad_D2.0mm -> hellen-one-common:USB-MINI-B-VERTICAL
- M1: value Module-motor-driver-0.1 -> Module-power_12and5V-0.3; footprint hellen-one-motor-driver-0.1:motor-driver -> hellen-one-power_12and5V-0.3:power_12and5V
- M3: value mega-mcu144-0.1 -> Module-vr-discrete-0.5; footprint hellen-one-mega-mcu144-0.1:mega-mcu144 -> hellen-one-vr-discrete-0.5:vr-discrete
- M5: value Module-knock-0.2 -> Module-motor-driver-0.1; footprint hellen-one-knock-0.2:knock -> hellen-one-motor-driver-0.1:motor-driver
- M6: value Module-output-0.3 -> Module-wbo-0.5; footprint hellen-one-output-0.3:output -> hellen-one-wbo-0.5:wbo
- M7: value Module-ign8-0.2 -> Module:mega-mcu100/0.3; footprint hellen-one-ign8-0.2:ign8 -> hellen-one-mega-mcu100-0.3:mega-mcu100
- M8: value Module-power_12and5V-0.1 -> Module-can-0.1; footprint hellen-one-power_12and5V-0.1:power_12and5V -> hellen-one-can-0.1:can
- P1: footprint hellen121vag:368255-2 -> footprints:368255-2
- P2: value Pad -> 368255-2; footprint hellen-one-common:PAD-TH -> footprints:368255-2
- R10, R11, R12: value Jumper-Pad-Pad -> 10k; footprint hellen-one-common:PAD-0805-PAD -> hellen-one-common:R0805
- R13: value Jumper-Pad-Pad -> 4.7k; footprint hellen-one-common:PAD-0805-PAD -> hellen-one-common:R0603
- R16, R17: value 5.1k -> 4.7k
- R2: value Jumper-Pad-Pad -> 33k; footprint hellen-one-common:PAD-0805-PAD -> hellen-one-common:R0603
- R20: value 1.6k -> 22
- R21: value 750 -> 22
- R23: footprint hellen-one-common:R0603 -> Resistor_SMD:R_2512_6332Metric
- R3: value Jumper-Pad-Pad -> 6.8k; footprint hellen-one-common:PAD-0805-PAD -> hellen-one-common:R0603
- R8, R9: value Jumper-Pad-Pad -> DNP; footprint hellen-one-common:PAD-0805-PAD -> hellen-one-common:R0805
- U3: value MCP6002-xSN -> VNLD5160TR-E
- moved R3 70.5 mm to (137.8, 33.0), turned to 0 degrees
- moved R2 68.7 mm to (137.8, 31.0), turned to 0 degrees
- moved F2 63.8 mm to (111.4, 63.3), turned to 0 degrees
- moved F1 62.0 mm to (111.4, 60.2), turned to 0 degrees
- moved R8 58.7 mm to (138.1, 43.5), turned to 0 degrees
- moved M6 58.0 mm to (83.4, 57.9)
- moved R9 54.6 mm to (138.1, 46.1), turned to 0 degrees
- moved M5 51.4 mm to (118.7, 67.6)
- moved M3 48.7 mm to (118.7, 16.3)
- moved P2 48.5 mm to (60.1, 33.0), turned to 0 degrees
- moved J1 47.7 mm to (121.4, 54.3)
- moved M1 47.5 mm to (118.7, 49.4)
- moved U3 45.6 mm to (114.5, 73.7), turned to 0 degrees
- moved R4 40.7 mm to (136.3, 63.1), turned to 0 degrees
- moved M8 39.7 mm to (83.4, 66.2)
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Connections:
- net /-ETB_OUT renamed PIN118
- D3 pad 1: /IN_VIGN -> PIN117
- D3 pad 2: Net-(D3-A) -> PIN16
- D4 pad 1: /IN_VIGN -> PIN117
- D4 pad 2: Net-(D3-A) -> PIN88
- D5 pad 1: +12V_RAW -> PIN43
- D5 pad 2: Net-(D5-A) -> PIN114
- D6 pad 1: +5V -> Net-(U2-T-)
- D6 pad 2: Net-(D6-K) -> Net-(U2-T+)
- F1 pad 1: Net-(F1-Pad1) -> PIN108
- F1 pad 2: +12V_RAW -> /IN_VIGN
- F2 pad 1: Net-(F2-Pad1) -> PIN120
- F2 pad 2: +12V_RAW -> PIN117
- J1 pad 2: /USBM -> /USB-
- J1 pad 3: /USBP -> /USB+
- J1 pad 4: unconnected-(J1-ID-Pad4) -> PIN114
- J1 pad 5: Net-(J1-GND) -> PIN114
- J2 pad 1: +12V_RAW -> /VBUS
- M1 pad S1: unconnected-(M1-12V_IN-PadS1) -> PIN114
- M3 pad E1: unconnected-(M3-SPI2_SCK-PadE1) -> /VR_DISCRETE_THR
- M3 pad E2: unconnected-(M3-SPI2_MISO-PadE2) -> /VR_DISCRETE_A
- M3 pad E3: unconnected-(M3-SPI2_MOSI-PadE3) -> /VR_DISCRETE
- M3 pad E4: unconnected-(M3-SPI2_CS-PadE4) -> +5VA
- M3 pad G: GND -> PIN114
- M3 pad W1: /IGN8 -> PIN18
- M3 pad W2: /IGN7 -> PIN17
- M5 pad W1: /IN_KNOCK1_RAW -> DC1_DIS_W1
- M5 pad W2: /VREF2 -> /DC1_PWM
- M6 pad G: GND -> PIN114
- M6 pad W1: /OUT_VVT1_2 -> +5VA
- M6 pad W2: /OUT_VVT1_2 -> unconnected-(M6-CAN_VIO-PadW2)
- M6 pad W3: /OUT_CHECK_ENGINE -> PIN83
- M6 pad W4: /OUT_WASTEGATE -> PIN82
- M6 pad W5: +12V_PROT -> unconnected-(M6-nReset-PadW5)
- M6 pad W6: /OUT_TACH -> unconnected-(M6-SWDIO-PadW6)
- M6 pad W7: /OUT_INJ4 -> unconnected-(M6-SWCLK-PadW7)
- M6 pad W9: Net-(M6C-OUT_LOW7_PULLUP) -> unconnected-(M6-VDDA-PadW9)
- M7 pad G: GND -> PIN114
- M7 pad S1: /OUT_IGN8 -> PIN89
- M7 pad S2: /OUT_IGN7 -> PIN34
- M7 pad S3: /OUT_IGN6 -> PIN35
- M7 pad S4: /OUT_IGN5 -> PIN36
- M7 pad S5: /OUT_IGN4 -> unconnected-(M7-VREF2-PadS5)
- M7 pad S6: /OUT_IGN3 -> /IN_VMAIN
- M7 pad S7: /OUT_IGN2 -> /IN_AUX3
- M7 pad S8: /OUT_IGN1 -> PIN91
- M8 pad E1: /VBAT -> PIN114
- M8 pad S1: GND -> unconnected-(M8-CANL-PadS1)
- M8 pad V1: /V12_PERM -> +5VA
- M8 pad V2: /IN_VIGN -> +3.3VA
- P1 pad 1: GND -> PIN1
- P1 pad 10: Net-(P10-Pin_1) -> (no net)
- P1 pad 100: unconnected-(P1-Pad100) -> (no net)
- P1 pad 101: /IN_MAP2 -> (no net)
- P1 pad 102: /OUT_IGN1 -> (no net)
- P1 pad 103: /OUT_IGN5 -> (no net)
- P1 pad 104: /OUT_WASTEGATE -> (no net)
- P1 pad 105: /OUT_IDLE -> (no net)
- P1 pad 106: /IN_KNOCK1_RAW -> (no net)
- P1 pad 107: unconnected-(P1-Pad107) -> (no net)
- P1 pad 108: GNDA -> (no net)
- P1 pad 109: unconnected-(P1-Pad109) -> (no net)
- P1 pad 11: Net-(P11-Pin_1) -> (no net)
- P1 pad 110: /OUT_IGN6 -> (no net)
- P1 pad 111: /OUT_IGN3 -> (no net)
- P1 pad 112: /OUT_INJ6 -> (no net)
- P1 pad 113: /OUT_INJ5 -> (no net)
- P1 pad 114: unconnected-(P1-Pad114) -> PIN114
- P1 pad 115: /OUT_VVT1_2 -> PIN114
- P1 pad 116: unconnected-(P1-Pad116) -> PIN116
- P1 pad 117: /+ETB_OUT -> PIN117
- P1 pad 119: unconnected-(P1-Pad119) -> PIN119
- P1 pad 12: Net-(P12-Pin_1) -> (no net)
- P1 pad 120: /OUT_VVT2_B2 -> PIN120
- P1 pad 121: Net-(F2-Pad1) -> PIN121
- P1 pad 13: Net-(P13-Pin_1) -> (no net)
- P1 pad 14: /IN_AFR -> (no net)
- P1 pad 15: unconnected-(P1-Pad15) -> (no net)
- P1 pad 16: unconnected-(P1-Pad16) -> (no net)
- P1 pad 17: Net-(P17-Pin_1) -> (no net)
- P1 pad 18: /OUT_VVT2_B1 -> (no net)
- P1 pad 19: /OUT_INJ7 -> (no net)
- P1 pad 2: GND -> PIN2
- P1 pad 20: Net-(P20-Pin_1) -> (no net)
- P1 pad 21: Net-(P1-Pad21) -> (no net)
- P1 pad 22: /OUT_VVT1_1 -> (no net)
- P1 pad 23: Net-(P1-Pad23) -> (no net)
- P1 pad 24: /OUT_INJ8 -> (no net)
- P1 pad 25: unconnected-(P1-Pad25) -> (no net)
- P1 pad 26: /IN_IAT -> (no net)
- P1 pad 27: GNDA -> (no net)
- P1 pad 28: Net-(P28-Pin_1) -> (no net)
- P1 pad 29: /IN_MAF -> (no net)
- P1 pad 3: Net-(F1-Pad1) -> PIN114
- P1 pad 30: unconnected-(P1-Pad30) -> (no net)
- P1 pad 31: unconnected-(P1-Pad31) -> (no net)
- P1 pad 32: GND -> (no net)
- P1 pad 33: GNDA -> (no net)
- P1 pad 34: /IN_PPS1 -> (no net)
- P1 pad 35: /IN_PPS2 -> (no net)
- P1 pad 36: GNDA -> (no net)
- P1 pad 37: Net-(P1-Pad37) -> (no net)
- P1 pad 38: /IN_RES1 -> (no net)
- P1 pad 39: /IN_RES2 -> (no net)
- P1 pad 4: unconnected-(P1-Pad4) -> PIN4
- P1 pad 40: Net-(P40-Pin_1) -> (no net)
- P1 pad 41: Net-(P41-Pin_1) -> (no net)
- P1 pad 42: unconnected-(P1-Pad42) -> (no net)
- P1 pad 43: Net-(P43-Pin_1) -> (no net)
- P1 pad 44: Net-(P44-Pin_1) -> (no net)
- P1 pad 45: Net-(P45-Pin_1) -> (no net)
- P1 pad 46: Net-(P46-Pin_1) -> (no net)
- P1 pad 47: /OUT_CHECK_ENGINE -> (no net)
- P1 pad 48: Net-(P48-Pin_1) -> (no net)
- P1 pad 49: Net-(P49-Pin_1) -> (no net)
- P1 pad 5: /LSU_HEAT- -> PIN5
- P1 pad 50: GNDA -> (no net)
- P1 pad 51: Net-(P1-Pad51) -> (no net)
- P1 pad 52: Net-(P1-Pad52) -> (no net)
- P1 pad 53: +5VP -> (no net)
- P1 pad 54: /IN_VSS -> (no net)
- P1 pad 55: /IN_D1 -> (no net)
- P1 pad 56: Net-(P56-Pin_1) -> (no net)
- P1 pad 57: /IN_D2 -> (no net)
- P1 pad 58: /CAN- -> (no net)
- P1 pad 59: GND -> (no net)
- P1 pad 6: unconnected-(P1-Pad6) -> (no net)
- P1 pad 60: /CAN+ -> (no net)
- P1 pad 61: Net-(P61-Pin_1) -> (no net)
- P1 pad 62: /V12_PERM -> (no net)
- P1 pad 63: Net-(P63-Pin_1) -> (no net)
- P1 pad 64: Net-(P64-Pin_1) -> (no net)
- P1 pad 65: /OUT_FUEL_PUMP_RELAY -> (no net)
- P1 pad 66: Net-(P66-Pin_1) -> (no net)
- P1 pad 67: Net-(P67-Pin_1) -> (no net)
- P1 pad 68: Net-(P68-Pin_1) -> (no net)
- P1 pad 69: Net-(P69-Pin_1) -> (no net)
- P1 pad 7: /OUT_IGN2 -> (no net)
- P1 pad 70: Net-(P1-Pad70) -> (no net)
- P1 pad 71: Net-(P1-Pad71) -> (no net)
- P1 pad 72: +5VP -> (no net)
- P1 pad 73: +5VP -> (no net)
- P1 pad 74: Net-(P74-Pin_1) -> (no net)
- P1 pad 75: /IN_D3 -> (no net)
- P1 pad 76: /IN_D4 -> (no net)
- P1 pad 77: unconnected-(P1-Pad77) -> (no net)
- P1 pad 78: unconnected-(P1-Pad78) -> (no net)
- P1 pad 79: unconnected-(P1-Pad79) -> (no net)
- P1 pad 8: /OUT_IGN7 -> (no net)
- P1 pad 80: Net-(P80-Pin_1) -> (no net)
- P1 pad 81: /OUT_FUEL_CONSUM -> (no net)
- P1 pad 82: /IN_CRANK+ -> (no net)
- P1 pad 83: +5VP -> (no net)
- P1 pad 84: /IN_TPS2 -> (no net)
- P1 pad 85: /IN_IAT -> (no net)
- P1 pad 86: /IN_CAM1 -> (no net)
- P1 pad 87: /IN_CAM2 -> (no net)
- P1 pad 88: /OUT_INJ4 -> (no net)
- P1 pad 89: /OUT_INJ2 -> (no net)
- P1 pad 9: Net-(P9-Pin_1) -> (no net)
- P1 pad 90: /IN_CRANK- -> (no net)
- P1 pad 91: GNDA -> (no net)
- P1 pad 92: /IN_TPS1 -> (no net)
- P1 pad 93: /IN_CLT -> (no net)
- P1 pad 94: /OUT_IGN4 -> (no net)
- P1 pad 95: /OUT_IGN8 -> (no net)
- P1 pad 96: /OUT_INJ1 -> (no net)
- P1 pad 97: /OUT_INJ3 -> (no net)
- P1 pad 98: +5VP -> (no net)
- P1 pad 99: GNDA -> (no net)
- P2 pad 1: /IN_A1 -> (no net)
- R10 pad 1: Net-(P1-Pad51) -> PIN113
- R10 pad 2: /LSU_SENSOR_U/PUMP_I -> PIN84
- R11 pad 1: Net-(P1-Pad52) -> PIN113
- R11 pad 2: /LSU_PUMP_I -> PIN85
- R12 pad 1: Net-(P1-Pad70) -> PIN113
- R12 pad 2: /LSU_SENSOR_U -> PIN89
- R13 pad 1: Net-(P1-Pad71) -> Net-(M7-LED_GREEN)
- R13 pad 2: /LSU_CALIBR_RES -> PIN114
- R16 pad 1: Net-(D3-A) -> /LS_HOT2
- R16 pad 2: GND -> PIN114
- R17 pad 1: Net-(D5-A) -> /LS_HOT1
- R17 pad 2: GND -> Net-(U3-IN2)
- R2 pad 1: Net-(P1-Pad21) -> /IN_VMAIN
- R2 pad 2: /OUT_MAIN_RELAY -> PIN120
- R20 pad 1: Net-(D6-K) -> Net-(Q3-G)
- R20 pad 2: GND -> Net-(F5-Pad1)
- R21 pad 2: GND -> Net-(F6-Pad1)
- R23 pad 1: Net-(J1-GND) -> Net-(F5-Pad1)
- R23 pad 2: GND -> PIN12
- R3 pad 1: /OUT_MAIN_RELAY -> PIN114
- R3 pad 2: Net-(P1-Pad23) -> /IN_VMAIN
- R4 pad 1: Net-(P1-Pad37) -> Net-(M1-PG_5VP)
- R4 pad 2: /OUT_TACH -> /PG_5VP
- R8 pad 1: /IN_VIGN -> PIN85
- R8 pad 2: Net-(P1-Pad21) -> +5VA
- R9 pad 1: Net-(F1-Pad1) -> PIN89
- R9 pad 2: /IN_VIGN -> +5VA
- U3 pad 1: Net-(U3A--) -> Net-(U3-IN1)
- U3 pad 2: Net-(U3A--) -> unconnected-(U3-STATUS1-Pad2)
- U3 pad 3: /IN_KNOCK1 -> Net-(U3-IN2)
- U3 pad 4: GND -> unconnected-(U3-STATUS2-Pad4)
- U3 pad 5: GND -> PIN114
- U3 pad 6: Net-(U3B--) -> PIN86
- U3 pad 7: Net-(U3B--) -> PIN114
- U3 pad 8: +5V -> PIN87
Routing:
- net +12V_RAW: track 450.9 -> 0.00 mm, vias 10 -> 0
- net PIN113: track 0.00 -> 346.8 mm, vias 0 -> 1
- net (no net): track 41.0 -> 387.0 mm, vias 2 -> 3
- net +5V: track 301.1 -> 0.00 mm, vias 3 -> 0
- net PIN114: track 0.00 -> 263.1 mm, vias 0 -> 45
- net PIN106: track 0.00 -> 213.3 mm, vias 0 -> 1
- net +3V3: track 198.6 -> 0.00 mm, vias 4 -> 0
- net /OUT_IGN1: track 181.1 -> 0.00 mm, vias 2 -> 0
- net /OUT_IGN3: track 177.7 -> 0.00 mm, vias 2 -> 0
- net /OUT_IGN5: track 173.6 -> 0.00 mm, vias 1 -> 0
- net /OUT_IGN6: track 172.1 -> 0.00 mm, vias 2 -> 0
- net /OUT_IGN4: track 171.5 -> 0.00 mm, vias 2 -> 0
- net /OUT_IGN8: track 161.5 -> 0.00 mm, vias 1 -> 0
- net Net-(F1-Pad1): track 156.2 -> 0.00 mm, vias 1 -> 0
- net /OUT_IGN2: track 155.4 -> 0.00 mm, vias 2 -> 0
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- added copper zone on B.Cu, net PIN114
- added copper zone on F.Cu, net PIN114
- removed copper zone on B.Cu, net /OUT_INJ2
- removed copper zone on B.Cu, net GND
- removed copper zone on F.Cu, net GND
- removed copper zone on B.Cu, net Net-(J1-GND)
- removed copper zone on F.Cu, net Net-(J1-GND)
Other:
- board text removed: "12V SRC"
- board text removed: "<- Knock audio"
- board text removed: "G"
- board text removed: "PROG"
