File: hellen121vag.kicad_pcb (KiCad board)
At the start: 4 copper layers, 164 x 118 mm, 100 parts, among them J1 Conn_01x05_Male, J2 USB_B_Mini, M1 Module-power_12and5V-0.3, M2 Module-knock-0.2, M3 Module-vr-discrete-0.5, M4 Module-vr-max9924-0.1, M5 Module-motor-driver-0.1, M6 Module-wbo-0.5, M7 Module:mega-mcu100/0.3, M8 Module-can-0.1, P1 368255-2, P2 368255-2, Q1 AO3400A, Q2 ISL9V3040D3ST, Q3 ISL9V3040D3ST, Q4 ISL9V3040D3ST, Q5 ISL9V3040D3ST, Q6 ISL9V3040D3ST, Q7 ISL9V3040D3ST, U1 BTS6143D, U2 MAX31855KASA, U3 VNLD5160TR-E, U4 VNLD5160TR-E, U5 VNLD5160TR-E, U6 VNLD5160TR-E, U7 VNLD5160TR-E, U8 VNLD5160TR-E

Commit message: wq
Parts:
- removed C1, C3: 10n, hellen-one-common:C0603
- removed C2, C4: 100n, hellen-one-common:C0603
- removed C5: 1u, hellen-one-common:C0603
- removed F4: 50mA, Fuse:Fuse_0603_1608Metric
- removed G***: LOGO, hellen-one-common:LOGO
- removed J1: Conn_01x05_Male, Connector_Molex:Molex_SPOX_5267-05A_1x05_P2.50mm_Vertical
- removed J2: USB_B_Mini, hellen-one-common:USB-MINI-B-VERTICAL
- removed U1: BTS6143D, Package_TO_SOT_SMD:TO-252-4
- removed U2: MAX31855KASA, Package_SO:SOIC-8_3.9x4.9mm_P1.27mm
- added C28: 10n, hellen-one-common:C0603, F.Cu at (171.0, 61.8)
- added C29: 100n, hellen-one-common:C0603, F.Cu at (173.3, 54.3)
- added C30: 10n, hellen-one-common:C0603, F.Cu at (173.1, 60.8)
- added C31: 100n, hellen-one-common:C0603, F.Cu at (174.3, 50.3)
- added C32: 1u, hellen-one-common:C0603, F.Cu at (175.8, 50.3)
- added F10: 50mA, Fuse:Fuse_0603_1608Metric, B.Cu at (165.8, 55.3)
- added J21: Conn_01x05_Male, Connector_Molex:Molex_SPOX_5267-05A_1x05_P2.50mm_Vertical, F.Cu at (173.8, 5.62)
- added J22: USB_B_Mini, hellen-one-common:USB-MINI-B-VERTICAL, F.Cu at (157.3, 7.62)
- added R51: 4.7k, hellen-one-common:R0603, B.Cu at (136.3, 47.8)
- added R52: 4.7k, hellen-one-common:R0603, B.Cu at (187.8, 15.3)
- added R53: 4.7k, hellen-one-common:R0603, B.Cu at (184.8, 15.3)
- added R54: 1k, hellen-one-common:R0603, F.Cu at (62.8, 67.8)
- added U10: BTS6143D, Package_TO_SOT_SMD:TO-252-4, F.Cu at (64.8, 77.1)
- added U11: VNLD5160TR-E, Package_SO:SOIC-8_3.9x4.9mm_P1.27mm, F.Cu at (185.3, 21.3)
- added U9: VNLD5160TR-E, Package_SO:SOIC-8_3.9x4.9mm_P1.27mm, F.Cu at (124.8, 49.8)
- D1, D2, D3, D4, F5, F6, F7, F8, F9, R13, R16, R19, R2, R22, R25, R28, R3, R31, R32, R33, R34, R35, R36, R37, R38, R39, R40, R41, R42, R43, R44, R45, R46, R47, R48, R49, R50: moved to B.Cu
- M5: value Module-motor-driver-0.1 -> Module-wbo-0.5; footprint hellen-one-motor-driver-0.1:motor-driver -> hellen-one-wbo-0.5:wbo
- M6: value Module-wbo-0.5 -> Module:mega-mcu100/0.3; footprint hellen-one-wbo-0.5:wbo -> hellen-one-mega-mcu100-0.3:mega-mcu100
- M7: value Module:mega-mcu100/0.3 -> Module-can-0.1; footprint hellen-one-mega-mcu100-0.3:mega-mcu100 -> hellen-one-can-0.1:can
- M8: value Module-can-0.1 -> Module-motor-driver-0.1; footprint hellen-one-can-0.1:can -> hellen-one-motor-driver-0.1:motor-driver
- Q1: value AO3400A -> ISL9V3040D3ST; footprint Package_TO_SOT_SMD:SOT-23 -> Package_TO_SOT_SMD:TO-252-2
- Q7: value ISL9V3040D3ST -> AO3400A; footprint Package_TO_SOT_SMD:TO-252-2 -> Package_TO_SOT_SMD:SOT-23
- R14: value 1k -> 4.7k; moved to B.Cu
- R17, R18: value 4.7k -> 22; moved to B.Cu
- R20, R21, R26, R27: value 22 -> 0; footprint hellen-one-common:R0603 -> Resistor_SMD:R_2512_6332Metric; moved to B.Cu
- R23, R24: value 0 -> 22; footprint Resistor_SMD:R_2512_6332Metric -> hellen-one-common:R0603; moved to B.Cu
- R29, R30: value 0 -> 4.7k; footprint Resistor_SMD:R_2512_6332Metric -> hellen-one-common:R0603; moved to B.Cu
- U8: value VNLD5160TR-E -> MAX31855KASA
- moved D6 118.0 mm to (173.3, 57.3), turned to 90 degrees
- moved R13 107.9 mm to (157.3, 47.8)
- moved M7 95.3 mm to (173.3, 10.9), turned to 180 degrees
- moved Q7 88.2 mm to (65.8, 67.8), turned to -90 degrees
- moved L1 85.7 mm to (172.8, 65.3), turned to 90 degrees
- moved R21 85.1 mm to (133.3, 62.3), turned to -90 degrees
- moved L2 84.1 mm to (170.8, 65.3), turned to 90 degrees
- moved R16 83.7 mm to (131.8, 47.8), turned to -90 degrees
- moved R17 80.5 mm to (124.8, 57.3)
- moved R20 78.8 mm to (125.3, 62.2), turned to -90 degrees
- moved D3 75.6 mm to (125.8, 51.9), turned to -90 degrees
- moved D4 74.3 mm to (123.3, 51.8), turned to -90 degrees
- moved U8 70.8 mm to (170.3, 48.8), turned to 90 degrees
- moved F1 66.9 mm to (178.3, 63.8), turned to 90 degrees
- moved F2 64.3 mm to (175.8, 63.8), turned to 90 degrees
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Connections:
- D6 pad 1: Net-(U2-T-) -> (no net)
- D6 pad 2: Net-(U2-T+) -> (no net)
- F5 pad 2: /IGN2 -> /IGN1
- F6 pad 2: /IGN3 -> /IGN2
- F7 pad 2: /IGN4 -> /IGN3
- F8 pad 2: /IGN5 -> /IGN4
- F9 pad 2: /IGN6 -> /IGN5
- L1 pad 2: Net-(U2-T+) -> (no net)
- L2 pad 2: Net-(U2-T-) -> (no net)
- M5 pad W1: DC1_DIS_W1 -> +5VA
- M5 pad W2: /DC1_PWM -> (no net)
- M5 pad W3: unconnected-(M5-SCLK-PadW3) -> PIN83
- M5 pad W4: /DC1_DIR -> PIN82
- M5 pad W5: +3.3V -> (no net)
- M5 pad W6: unconnected-(M5-MISO-PadW6) -> (no net)
- M5 pad W7: unconnected-(M5-~CS-PadW7) -> (no net)
- M6 pad E1: PIN105 -> +5VA
- M6 pad E2: PIN104 -> (no net)
- M6 pad E3: PIN103 -> (no net)
- M6 pad E4: PIN102 -> (no net)
- M6 pad E5: PIN119 -> /VIGN
- M6 pad E6: PIN114 -> E6INJ7CANRX
- M6 pad W1: +5VA -> PIN113
- M6 pad W2: unconnected-(M6-CAN_VIO-PadW2) -> +5VA
- M6 pad W3: PIN83 -> /LS_HOT2
- M6 pad W4: PIN82 -> /LS_HOT1
- M6 pad W5: unconnected-(M6-nReset-PadW5) -> /IGN6
- M6 pad W6: unconnected-(M6-SWDIO-PadW6) -> /IGN5
- M6 pad W7: unconnected-(M6-SWCLK-PadW7) -> /IGN4
- M6 pad W8: unconnected-(M6-V33_OUT-PadW8) -> /IGN3
- M6 pad W9: unconnected-(M6-VDDA-PadW9) -> /IGN2
- M7 pad E1: +5VA -> PIN114
- M7 pad S1: PIN89 -> (no net)
- M7 pad S2: PIN34 -> (no net)
- M8 pad S1: unconnected-(M8-CANL-PadS1) -> Net-(F3-Pad2)
- M8 pad S2: unconnected-(M8-CANH-PadS2) -> PIN2
- Q1 pad 1: Net-(M7-LED_GREEN) -> (no net)
- Q1 pad 2: PIN114 -> PIN13
- Q1 pad 3: Net-(Q1-D) -> PIN114
- Q2 pad 2: PIN13 -> PIN12
- Q3 pad 2: PIN12 -> PIN10
- Q4 pad 2: PIN10 -> PIN9
- Q5 pad 2: PIN9 -> PIN11
- Q6 pad 2: PIN11 -> PIN8
- Q7 pad 1: Net-(Q7-G) -> (no net)
- Q7 pad 2: PIN8 -> PIN114
- Q7 pad 3: PIN114 -> (no net)
- R13 pad 1: Net-(M7-LED_GREEN) -> /LS_HOT2
- R13 pad 2: PIN114 -> Net-(U7-IN1)
- R14 pad 1: Net-(U1-IS) -> /LS_HOT1
- R14 pad 2: PIN114 -> Net-(U7-IN2)
- R15 pad 1: /LS_HOT2 -> (no net)
- R15 pad 2: Net-(U3-IN1) -> PIN114
- R16 pad 1: /LS_HOT2 -> /LS1
- R17 pad 1: /LS_HOT1 -> (no net)
- R17 pad 2: Net-(U3-IN2) -> Net-(F5-Pad1)
- R18 pad 1: /LS_HOT1 -> Net-(Q2-G)
- R18 pad 2: PIN114 -> Net-(F6-Pad1)
- R19 pad 1: Net-(Q2-G) -> Net-(Q3-G)
- R19 pad 2: Net-(F4-Pad1) -> Net-(F7-Pad1)
- R20 pad 1: Net-(Q3-G) -> Net-(F5-Pad1)
- R20 pad 2: Net-(F5-Pad1) -> PIN13
- R21 pad 1: Net-(Q4-G) -> Net-(F6-Pad1)
- R21 pad 2: Net-(F6-Pad1) -> PIN12
- R22 pad 1: Net-(F4-Pad1) -> Net-(F7-Pad1)
- R22 pad 2: PIN13 -> PIN10
- R23 pad 1: Net-(F5-Pad1) -> Net-(Q4-G)
- R23 pad 2: PIN12 -> Net-(F8-Pad1)
- R24 pad 1: Net-(F6-Pad1) -> Net-(Q5-G)
- R24 pad 2: PIN10 -> Net-(F9-Pad1)
- R25 pad 1: Net-(Q5-G) -> Net-(Q6-G)
- R25 pad 2: Net-(F7-Pad1) -> (no net)
- R26 pad 1: Net-(Q6-G) -> Net-(F8-Pad1)
- R26 pad 2: Net-(F8-Pad1) -> PIN9
- R27 pad 1: Net-(Q7-G) -> Net-(F9-Pad1)
- R27 pad 2: Net-(F9-Pad1) -> PIN11
- R28 pad 1: Net-(F7-Pad1) -> (no net)
- R28 pad 2: PIN9 -> PIN8
- R29 pad 1: Net-(F8-Pad1) -> /INJ1
- R29 pad 2: PIN11 -> PIN114
- R30 pad 1: Net-(F9-Pad1) -> /INJ3
- R30 pad 2: PIN8 -> PIN114
- R31 pad 1: E6INJ7CANRX -> /INJ5
- R31 pad 2: Net-(U4-IN1) -> PIN114
- R32 pad 1: E7INJ8CANTX -> /INJ2
- R32 pad 2: Net-(U4-IN2) -> PIN114
- R33 pad 1: E7INJ8CANTX -> /INJ4
- R34 pad 1: E6INJ7CANRX -> /INJ6
- R35 pad 1: /INJ1 -> /LS_HOT1
- R36 pad 1: /INJ1 -> /LS_HOT2
- R36 pad 2: Net-(U7-IN1) -> PIN114
- R37 pad 1: /INJ2 -> /LS3
- R38 pad 1: /INJ2 -> /LS2
- R38 pad 2: Net-(U7-IN2) -> PIN114
- R39 pad 1: /INJ3 -> /LS4
- R40 pad 1: /INJ3 -> E6INJ7CANRX
- R40 pad 2: Net-(U5-IN1) -> PIN114
- R41 pad 1: /INJ4 -> E7INJ8CANTX
- R41 pad 2: Net-(U5-IN2) -> PIN114
- R42 pad 1: /INJ4 -> /LS3
- R42 pad 2: PIN114 -> (no net)
- R43 pad 1: /INJ5 -> /LS4
- R43 pad 2: Net-(U6-IN1) -> (no net)
- R44 pad 1: /INJ5 -> /LS1
- R44 pad 2: PIN114 -> Net-(U3-IN1)
- R45 pad 1: /INJ6 -> /LS2
- R45 pad 2: PIN114 -> Net-(U3-IN2)
- R46 pad 1: /INJ6 -> /INJ1
- R46 pad 2: Net-(U6-IN2) -> Net-(U4-IN1)
- R47 pad 1: /LS2 -> /INJ2
- R47 pad 2: Net-(U8-IN1) -> Net-(U4-IN2)
- R48 pad 1: /LS2 -> /INJ3
- R48 pad 2: PIN114 -> Net-(U5-IN1)
- R49 pad 1: /LS1 -> /INJ4
- R49 pad 2: Net-(U8-IN2) -> Net-(U5-IN2)
- R50 pad 1: /LS1 -> /INJ5
- R50 pad 2: PIN114 -> Net-(U6-IN1)
- U3 pad 6: PIN86 -> PIN15
- U3 pad 8: PIN87 -> PIN14
- U4 pad 6: PIN51 -> PIN45
- U4 pad 8: PIN50 -> PIN44
- U7 pad 6: PIN45 -> PIN86
- U7 pad 8: PIN44 -> PIN87
- U8 pad 1: Net-(U8-IN1) -> PIN114
- U8 pad 2: unconnected-(U8-STATUS1-Pad2) -> (no net)
- U8 pad 3: Net-(U8-IN2) -> (no net)
- U8 pad 4: unconnected-(U8-STATUS2-Pad4) -> +3.3VA
- U8 pad 5: PIN114 -> /SCK3
- U8 pad 6: PIN14 -> /EGT/SPI_CS
- U8 pad 7: PIN114 -> /MISO3
- U8 pad 8: PIN15 -> (no net)
Routing:
- net (no net): track 387.0 -> 0.00 mm, vias 3 -> 0
- net PIN113: track 346.8 -> 0.00 mm, vias 1 -> 0
- net PIN114: track 263.1 -> 0.00 mm, vias 45 -> 31
- net PIN106: track 213.3 -> 0.00 mm, vias 1 -> 0
- net PIN102: track 118.2 -> 0.00 mm, vias 1 -> 0
- net PIN18: track 117.6 -> 0.00 mm
- net PIN111: track 115.4 -> 0.00 mm, vias 1 -> 0
- net PIN103: track 111.9 -> 0.00 mm
- net PIN110: track 110.9 -> 0.00 mm, vias 1 -> 0
- net PIN6: track 110.9 -> 0.00 mm
- net PIN94: track 109.5 -> 0.00 mm, vias 1 -> 0
- net PIN81: track 104.5 -> 0.00 mm, vias 2 -> 0
- net GNDA: track 104.1 -> 0.00 mm, vias 1 -> 0
- net PIN95: track 101.1 -> 0.00 mm
- net PIN7: track 92.6 -> 0.00 mm, vias 1 -> 0
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Other:
- board text removed: "+12"
- board text removed: "+3.3"
- board text removed: "+5"
- board text removed: "3.3"
- board text removed: "Always looking for C/C++/PHP/Java developers https://rusefi.com/s/mission"
- board text removed: "Baro"
- board text removed: "CLK"
- board text removed: "DIO"
- board text removed: "GND"
- board text removed: "Hellen121vag"
- board text removed: "RESET"
- board text removed: "RST"
- board text removed: "SWD WBO"
- board text removed: "Vign"
- board text removed: "http://rusefi.com/s/hellen121vag"
- board text removed: "rev. d"
- board text removed: "© andreika, 2021"
