File: INJ6.kicad_sch (KiCad schematic)
At the start: 20 parts, among them U4 VNLD5160TR-E, U5 VNLD5160TR-E, U6 VNLD5160TR-E, U7 VNLD5160TR-E

Commit message: wwew
Parts:
- renumbered R31 to R30, R32 to R31, R33 to R32, R34 to R33, R35 to R34, R36 to R35, R37 to R36, R38 to R37, R39 to R38, R40 to R39, R41 to R40, R42 to R41, R43 to R42, R44 to R43, R45 to R44, R46 to R45, U4 to U2, U5 to U3, U6 to U4, U7 to U5
