File: LS4.kicad_sch (KiCad schematic)
At the start: 5 parts, among them U8 VNLD5160TR-E

Commit message: awsw
Parts:
- U8: value VNLD5160TR-E -> MAX31855KASA; LCSC C377942 -> C52028
Changed lines of the file:
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@@
+	(wire
+		(pts
+			(xy 146.05 78.74) (xy 157.48 78.74)
+		)
+		(stroke
+			(width 0)
+			(type default)
+		)
+	)
 	(wire
 		(pts
@@
 		(pts
 			(xy 146.05 83.82) (xy 157.48 83.82)
-		)
-		(stroke
-			(width 0)
-			(type default)
-		)
-	)
-	(wire
-		(pts
-			(xy 146.05 78.74) (xy 157.48 78.74)
 		)
 		(stroke
@@
 			)
 		)
-		(property "Value" "VNLD5160TR-E"
+		(property "Value" "MAX31855KASA"
 			(at 132.08 73.66 0)
 			(effects
@@
 			)
 		)
-		(property "Datasheet" ""
+		(property "Datasheet" "http://datasheets.maximintegrated.com/en/ds/MAX31855.pdf"
 			(at 146.05 78.74 0)
 			(effects
@@
 			)
 		)
-		(property "LCSC" "C377942"
+		(property "LCSC" "C52028"
 			(at 134.62 81.28 0)
 			(effects

Commit message: wwew
Parts:
- renumbered R47 to R13, R48 to R14, R49 to R16, R50 to R17, U8 to U1
Changed lines of the file:
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@@
 		(on_board yes)
 		(dnp no)
-		(property "Reference" "R47"
+		(property "Reference" "R13"
 			(at 162.56 76.2 0)
 			(effects
@@
 		(instances
 			(project "hellen121vag"
-				(path "/45c1f041-3b7c-4036-abe9-e26621c05a73/5b484501-f65a-484d-a841-b73263bff7a2"
-					(reference "R47")
+				(path "/45c1f041-3b7c-4036-abe9-e26621c05a73/37c68176-bc6d-4360-9788-c5c46985dc55"
+					(reference "R13")
 					(unit 1)
 				)
@@
 		(on_board yes)
 		(dnp no)
-		(property "Reference" "#PWR080"
+		(property "Reference" "#PWR0102"
 			(at 115.57 95.25 0)
 			(effects
@@
 		(instances
 			(project "hellen121vag"
-				(path "/45c1f041-3b7c-4036-abe9-e26621c05a73/5b484501-f65a-484d-a841-b73263bff7a2"
-					(reference "#PWR080")
+				(path "/45c1f041-3b7c-4036-abe9-e26621c05a73/37c68176-bc6d-4360-9788-c5c46985dc55"
+					(reference "#PWR0102")
 					(unit 1)
 				)
@@
 		(on_board yes)
 		(dnp no)
-		(property "Reference" "R49"
+		(property "Reference" "R16"
 			(at 162.56 81.28 0)
 			(effects
@@
 		(instances
 			(project "hellen121vag"
-				(path "/45c1f041-3b7c-4036-abe9-e26621c05a73/5b484501-f65a-484d-a841-b73263bff7a2"
-					(reference "R49")
+				(path "/45c1f041-3b7c-4036-abe9-e26621c05a73/37c68176-bc6d-4360-9788-c5c46985dc55"
+					(reference "R16")
 					(unit 1)
 				)
@@
 		(dnp no)
 		(fields_autoplaced yes)
-		(property "Reference" "U8"
+		(property "Reference" "U1"
 			(at 132.08 71.12 0)
 			(effects
@@
 		(instances
 			(project "hellen121vag"
-				(path "/45c1f041-3b7c-4036-abe9-e26621c05a73/5b484501-f65a-484d-a841-b73263bff7a2"
-					(reference "U8")
+				(path "/45c1f041-3b7c-4036-abe9-e26621c05a73/37c68176-bc6d-4360-9788-c5c46985dc55"
+					(reference "U1")
 					(unit 1)
 				)
@@
 		(on_board yes)
 		(dnp no)
-		(property "Reference" "R50"
+		(property "Reference" "R17"
 			(at 165.1 88.9 0)
 			(effects
@@
 		(instances
 			(project "hellen121vag"
-				(path "/45c1f041-3b7c-4036-abe9-e26621c05a73/5b484501-f65a-484d-a841-b73263bff7a2"
-					(reference "R50")
+				(path "/45c1f041-3b7c-4036-abe9-e26621c05a73/37c68176-bc6d-4360-9788-c5c46985dc55"
+					(reference "R17")
 					(unit 1)
 				)
@@
 		(on_board yes)
 		(dnp no)
-		(property "Reference" "R48"
+		(property "Reference" "R14"
 			(at 165.1 73.66 0)
 			(effects
@@
 		(instances
 			(project "hellen121vag"
-				(path "/45c1f041-3b7c-4036-abe9-e26621c05a73/5b484501-f65a-484d-a841-b73263bff7a2"
-					(reference "R48")
+				(path "/45c1f041-3b7c-4036-abe9-e26621c05a73/37c68176-bc6d-4360-9788-c5c46985dc55"
+					(reference "R14")
 					(unit 1)
 				)
@@
 		(on_board yes)
 		(dnp no)
-		(property "Reference" "#PWR082"
+		(property "Reference" "#PWR0101"
 			(at 167.64 100.33 0)
 			(effects
@@
 		(instances
 			(project "hellen121vag"
-				(path "/45c1f041-3b7c-4036-abe9-e26621c05a73/5b484501-f65a-484d-a841-b73263bff7a2"
-					(reference "#PWR082")
+				(path "/45c1f041-3b7c-4036-abe9-e26621c05a73/37c68176-bc6d-4360-9788-c5c46985dc55"
+					(reference "#PWR0101")
 					(unit 1)
 				)
@@
 		(on_board yes)
 		(dnp no)
-		(property "Reference" "#PWR081"
+		(property "Reference" "#PWR0103"
 			(at 167.64 62.23 0)
 			(effects
@@
 		(instances
 			(project "hellen121vag"
-				(path "/45c1f041-3b7c-4036-abe9-e26621c05a73/5b484501-f65a-484d-a841-b73263bff7a2"
-					(reference "#PWR081")
-					(unit 1)
-				)
+				(path "/45c1f041-3b7c-4036-abe9-e26621c05a73/37c68176-bc6d-4360-9788-c5c46985dc55"
+					(reference "#PWR0103")
+					(unit 1)
+				)
