File: LS_HOT.kicad_sch (KiCad schematic)
At the start: 5 parts, among them U3 VNLD5160TR-E

Commit message: awsw
Parts:
- R15: LCSC C23162 -> C21189
- R17, R18: value 4.7k -> 22; LCSC C23162 -> C23345
Changed lines of the file:
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@@
 			)
 		)
-		(property "Value" "4.7k"
+		(property "Value" "22"
 			(at 168.91 85.09 0)
 			(effects
@@
 			)
 		)
-		(property "LCSC" "C23162"
+		(property "LCSC" "C23345"
 			(at 173.99 85.09 0)
 			(effects
@@
 			)
 		)
-		(property "LCSC" "C23162"
+		(property "LCSC" "C21189"
 			(at 173.99 80.01 0)
 			(effects
@@
 			)
 		)
-		(property "Value" "4.7k"
+		(property "Value" "22"
 			(at 173.99 90.17 0)
 			(effects
@@
 			)
 		)
-		(property "LCSC" "C23162"
-			(at 173.99 85.09 0)
-			(effects
+		(property "LCSC" "C23345"
+			(at 173.99 85.09 0)
+			(effects

Commit message: wwew
Parts:
- renumbered R15 to R46, R16 to R47, R17 to R48, R18 to R49, U3 to U6
Changed lines of the file:
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@@
 		(on_board yes)
 		(dnp no)
-		(property "Reference" "R17"
+		(property "Reference" "R48"
 			(at 168.91 82.55 0)
 			(effects
@@
 		(instances
 			(project "hellen121vag"
-				(path "/45c1f041-3b7c-4036-abe9-e26621c05a73/daaccf6d-1755-482f-b47d-8bf6bb55e029"
-					(reference "R17")
+				(path "/45c1f041-3b7c-4036-abe9-e26621c05a73/bdc55f5a-1abb-4701-b1a5-3e8a3596401f"
+					(reference "R48")
 					(unit 1)
 				)
@@
 		(on_board yes)
 		(dnp no)
-		(property "Reference" "#PWR061"
+		(property "Reference" "#PWR0123"
 			(at 173.99 101.6 0)
 			(effects
@@
 		(instances
 			(project "hellen121vag"
-				(path "/45c1f041-3b7c-4036-abe9-e26621c05a73/daaccf6d-1755-482f-b47d-8bf6bb55e029"
-					(reference "#PWR061")
+				(path "/45c1f041-3b7c-4036-abe9-e26621c05a73/bdc55f5a-1abb-4701-b1a5-3e8a3596401f"
+					(reference "#PWR0123")
 					(unit 1)
 				)
@@
 		(on_board yes)
 		(dnp no)
-		(property "Reference" "R15"
+		(property "Reference" "R46"
 			(at 168.91 77.47 0)
 			(effects
@@
 		(instances
 			(project "hellen121vag"
-				(path "/45c1f041-3b7c-4036-abe9-e26621c05a73/daaccf6d-1755-482f-b47d-8bf6bb55e029"
-					(reference "R15")
+				(path "/45c1f041-3b7c-4036-abe9-e26621c05a73/bdc55f5a-1abb-4701-b1a5-3e8a3596401f"
+					(reference "R46")
 					(unit 1)
 				)
@@
 		(dnp no)
 		(fields_autoplaced yes)
-		(property "Reference" "U3"
+		(property "Reference" "U6"
 			(at 138.43 72.39 0)
 			(effects
@@
 		(instances
 			(project "hellen121vag"
-				(path "/45c1f041-3b7c-4036-abe9-e26621c05a73/daaccf6d-1755-482f-b47d-8bf6bb55e029"
-					(reference "U3")
+				(path "/45c1f041-3b7c-4036-abe9-e26621c05a73/bdc55f5a-1abb-4701-b1a5-3e8a3596401f"
+					(reference "U6")
 					(unit 1)
 				)
@@
 		(on_board yes)
 		(dnp no)
-		(property "Reference" "#PWR060"
+		(property "Reference" "#PWR0122"
 			(at 173.99 63.5 0)
 			(effects
@@
 		(instances
 			(project "hellen121vag"
-				(path "/45c1f041-3b7c-4036-abe9-e26621c05a73/daaccf6d-1755-482f-b47d-8bf6bb55e029"
-					(reference "#PWR060")
+				(path "/45c1f041-3b7c-4036-abe9-e26621c05a73/bdc55f5a-1abb-4701-b1a5-3e8a3596401f"
+					(reference "#PWR0122")
 					(unit 1)
 				)
@@
 		(on_board yes)
 		(dnp no)
-		(property "Reference" "R16"
+		(property "Reference" "R47"
 			(at 171.45 74.93 0)
 			(effects
@@
 		(instances
 			(project "hellen121vag"
-				(path "/45c1f041-3b7c-4036-abe9-e26621c05a73/daaccf6d-1755-482f-b47d-8bf6bb55e029"
-					(reference "R16")
+				(path "/45c1f041-3b7c-4036-abe9-e26621c05a73/bdc55f5a-1abb-4701-b1a5-3e8a3596401f"
+					(reference "R47")
 					(unit 1)
 				)
@@
 		(on_board yes)
 		(dnp no)
-		(property "Reference" "#PWR059"
+		(property "Reference" "#PWR0124"
 			(at 121.92 96.52 0)
 			(effects
@@
 		(instances
 			(project "hellen121vag"
-				(path "/45c1f041-3b7c-4036-abe9-e26621c05a73/daaccf6d-1755-482f-b47d-8bf6bb55e029"
-					(reference "#PWR059")
+				(path "/45c1f041-3b7c-4036-abe9-e26621c05a73/bdc55f5a-1abb-4701-b1a5-3e8a3596401f"
+					(reference "#PWR0124")
 					(unit 1)
 				)
@@
 		(on_board yes)
 		(dnp no)
-		(property "Reference" "R18"
+		(property "Reference" "R49"
 			(at 171.45 90.17 0)
 			(effects
@@
 		(instances
 			(project "hellen121vag"
-				(path "/45c1f041-3b7c-4036-abe9-e26621c05a73/daaccf6d-1755-482f-b47d-8bf6bb55e029"
-					(reference "R18")
-					(unit 1)
-				)
+				(path "/45c1f041-3b7c-4036-abe9-e26621c05a73/bdc55f5a-1abb-4701-b1a5-3e8a3596401f"
+					(reference "R49")
+					(unit 1)
+				)
