File: egt.kicad_sch (KiCad schematic)
At the start: 9 parts, among them U2 MAX31855KASA

Commit message: wwew
Parts:
- renumbered U2 to U7
Changed lines of the file:
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@@
 		(instances
 			(project "hellen121vag"
-				(path "/45c1f041-3b7c-4036-abe9-e26621c05a73/475a7c51-3994-4e4b-a9a2-65181187b6d0"
+				(path "/45c1f041-3b7c-4036-abe9-e26621c05a73/6cde32b6-05f2-499d-9aff-ad44aab97055"
 					(reference "C1")
 					(unit 1)
@@
 		(on_board yes)
 		(dnp no)
-		(property "Reference" "#PWR057"
+		(property "Reference" "#PWR0128"
 			(at 143.51 55.88 0)
 			(effects
@@
 		(instances
 			(project "hellen121vag"
-				(path "/45c1f041-3b7c-4036-abe9-e26621c05a73/475a7c51-3994-4e4b-a9a2-65181187b6d0"
-					(reference "#PWR057")
+				(path "/45c1f041-3b7c-4036-abe9-e26621c05a73/6cde32b6-05f2-499d-9aff-ad44aab97055"
+					(reference "#PWR0128")
 					(unit 1)
 				)
@@
 		(instances
 			(project "hellen121vag"
-				(path "/45c1f041-3b7c-4036-abe9-e26621c05a73/475a7c51-3994-4e4b-a9a2-65181187b6d0"
+				(path "/45c1f041-3b7c-4036-abe9-e26621c05a73/6cde32b6-05f2-499d-9aff-ad44aab97055"
 					(reference "L1")
 					(unit 1)
@@
 		(instances
 			(project "hellen121vag"
-				(path "/45c1f041-3b7c-4036-abe9-e26621c05a73/475a7c51-3994-4e4b-a9a2-65181187b6d0"
+				(path "/45c1f041-3b7c-4036-abe9-e26621c05a73/6cde32b6-05f2-499d-9aff-ad44aab97055"
 					(reference "C2")
 					(unit 1)
@@
 		(on_board yes)
 		(dnp no)
-		(property "Reference" "U2"
+		(property "Reference" "U7"
 			(at 135.5441 52.07 0)
 			(effects
@@
 		(instances
 			(project "hellen121vag"
-				(path "/45c1f041-3b7c-4036-abe9-e26621c05a73/475a7c51-3994-4e4b-a9a2-65181187b6d0"
-					(reference "U2")
+				(path "/45c1f041-3b7c-4036-abe9-e26621c05a73/6cde32b6-05f2-499d-9aff-ad44aab97055"
+					(reference "U7")
 					(unit 1)
 				)
@@
 		(instances
 			(project "hellen121vag"
-				(path "/45c1f041-3b7c-4036-abe9-e26621c05a73/475a7c51-3994-4e4b-a9a2-65181187b6d0"
+				(path "/45c1f041-3b7c-4036-abe9-e26621c05a73/6cde32b6-05f2-499d-9aff-ad44aab97055"
 					(reference "D6")
 					(unit 1)
@@
 		(instances
 			(project "hellen121vag"
-				(path "/45c1f041-3b7c-4036-abe9-e26621c05a73/475a7c51-3994-4e4b-a9a2-65181187b6d0"
+				(path "/45c1f041-3b7c-4036-abe9-e26621c05a73/6cde32b6-05f2-499d-9aff-ad44aab97055"
 					(reference "L2")
 					(unit 1)
@@
 		(instances
 			(project "hellen121vag"
-				(path "/45c1f041-3b7c-4036-abe9-e26621c05a73/475a7c51-3994-4e4b-a9a2-65181187b6d0"
+				(path "/45c1f041-3b7c-4036-abe9-e26621c05a73/6cde32b6-05f2-499d-9aff-ad44aab97055"
 					(reference "C4")
 					(unit 1)
@@
 		(on_board yes)
 		(dnp no)
-		(property "Reference" "#PWR056"
+		(property "Reference" "#PWR0129"
 			(at 133.35 83.82 0)
 			(effects
@@
 		(instances
 			(project "hellen121vag"
-				(path "/45c1f041-3b7c-4036-abe9-e26621c05a73/475a7c51-3994-4e4b-a9a2-65181187b6d0"
-					(reference "#PWR056")
+				(path "/45c1f041-3b7c-4036-abe9-e26621c05a73/6cde32b6-05f2-499d-9aff-ad44aab97055"
+					(reference "#PWR0129")
 					(unit 1)
 				)
@@
 		(on_board yes)
 		(dnp no)
-		(property "Reference" "#PWR053"
+		(property "Reference" "#PWR0125"
 			(at 86.36 86.36 0)
 			(effects
@@
 		(instances
 			(project "hellen121vag"
-				(path "/45c1f041-3b7c-4036-abe9-e26621c05a73/475a7c51-3994-4e4b-a9a2-65181187b6d0"
-					(reference "#PWR053")
+				(path "/45c1f041-3b7c-4036-abe9-e26621c05a73/6cde32b6-05f2-499d-9aff-ad44aab97055"
+					(reference "#PWR0125")
 					(unit 1)
 				)
@@
 		(instances
 			(project "hellen121vag"
-				(path "/45c1f041-3b7c-4036-abe9-e26621c05a73/475a7c51-3994-4e4b-a9a2-65181187b6d0"
+				(path "/45c1f041-3b7c-4036-abe9-e26621c05a73/6cde32b6-05f2-499d-9aff-ad44aab97055"
 					(reference "C3")
 					(unit 1)
@@
 		(on_board yes)
 		(dnp no)
-		(property "Reference" "#PWR054"
+		(property "Reference" "#PWR0126"
 			(at 102.87 86.36 0)
 			(effects
@@
 		(instances
 			(project "hellen121vag"
-				(path "/45c1f041-3b7c-4036-abe9-e26621c05a73/475a7c51-3994-4e4b-a9a2-65181187b6d0"
-					(reference "#PWR054")
+				(path "/45c1f041-3b7c-4036-abe9-e26621c05a73/6cde32b6-05f2-499d-9aff-ad44aab97055"
+					(reference "#PWR0126")
 					(unit 1)
 				)
@@
 		(instances
 			(project "hellen121vag"
-				(path "/45c1f041-3b7c-4036-abe9-e26621c05a73/475a7c51-3994-4e4b-a9a2-65181187b6d0"
+				(path "/45c1f041-3b7c-4036-abe9-e26621c05a73/6cde32b6-05f2-499d-9aff-ad44aab97055"
 					(reference "C5")
 					(unit 1)
@@
 		(on_board yes)
 		(dnp no)
-		(property "Reference" "#PWR055"
+		(property "Reference" "#PWR0127"
 			(at 118.11 86.36 0)
 			(effects
@@
 		(instances
 			(project "hellen121vag"
-				(path "/45c1f041-3b7c-4036-abe9-e26621c05a73/475a7c51-3994-4e4b-a9a2-65181187b6d0"
-					(reference "#PWR055")
+				(path "/45c1f041-3b7c-4036-abe9-e26621c05a73/6cde32b6-05f2-499d-9aff-ad44aab97055"
+					(reference "#PWR0127")
 					(unit 1)
 				)
@@
 		(on_board yes)
 		(dnp no)
-		(property "Reference" "#PWR058"
+		(property "Reference" "#PWR0130"
 			(at 156.21 55.88 0)
 			(effects
@@
 		(instances
 			(project "hellen121vag"
-				(path "/45c1f041-3b7c-4036-abe9-e26621c05a73/475a7c51-3994-4e4b-a9a2-65181187b6d0"
-					(reference "#PWR058")
-					(unit 1)
-				)
+				(path "/45c1f041-3b7c-4036-abe9-e26621c05a73/6cde32b6-05f2-499d-9aff-ad44aab97055"
+					(reference "#PWR0130")
+					(unit 1)
+				)
