File: hellen121vag.kicad_sch (KiCad schematic)
At the start: 111 parts, among them J1 USB_B_Mini, J10 AudioJack_THR, J2 Conn_01x01, J3 Conn_01x01, J4 Conn_01x01, J5 Conn_01x01, J6 Conn_01x01, J7 Conn_01x08, J8 Conn_01x06, M11 Module-vr-discrete-0.4, M3 mega-mcu144-0.1, M5 Module-knock-0.2, M6 Module-output-0.3, M7 Module-ign8-0.2, M8 Module-power_12and5V-0.1, M9 Module-wbo-0.5, P1 368255-2, P10 Pad, P11 Pad, P12 Pad, P13 Pad, P14 Pad, P15 Pad, P16 Pad, P17 Pad, P2 Pad, P20 Pad, P28 Pad, P3 Pad, P4 Pad, P40 Pad, P41 Pad, P43 Pad, P44 Pad, P45 Pad, P46 Pad, P48 Pad, P49 Pad, P5 Pad, P56 Pad, P6 Pad, P61 Pad, P63 Pad, P64 Pad, P66 Pad, P67 Pad, P68 Pad, P69 Pad, P7 Pad, P74 Pad, P8 Pad, P80 Pad, P9 Pad, U1 L6205PD, U3 MCP6002-xSN

Commit message: weu
Parts:
- removed C1, C2: 100n, hellen-one-common:C0603, symbol hellen-one-common:Cap
- removed C10, C11, C12, C13, C14, C7, C8, C9: 10u, Capacitor_SMD:C_0805_2012Metric, symbol hellen-one-common:Cap
- removed C3: 220n, hellen-one-common:C0603, symbol hellen-one-common:Cap
- removed C4: 10n, hellen-one-common:C0603, symbol hellen-one-common:Cap
- removed C5: 5.6n, hellen-one-common:C0603, symbol hellen-one-common:Cap
- removed D1, D2: 1N4148WS, hellen-one-common:SOD-323, symbol hellen-one-common:1N4148WS
- removed R1: 100, hellen-one-common:R0603, symbol hellen-one-common:Res
- removed R22: 10k, hellen-one-common:R0603, symbol hellen-one-common:Res
- removed R5: 100k, hellen-one-common:R0603, symbol hellen-one-common:Res
- removed U1: L6205PD, hellen-one-common:SO20POWER, symbol hellen-one-common:L6205PD
- added M1: Module-motor-driver-0.1, hellen-one-motor-driver-0.1:motor-driver, symbol hellen-one-motor-driver-0.1:Module-motor-driver-0.1

Commit message: fg
Parts:
- removed BT1: BATTERY_CR2032, Battery:BatteryHolder_Keystone_1060_1x2032, symbol art-electro-power:BATTERY_CR2032
- removed C16: 100n, hellen-one-common:C0603, symbol hellen-one-common:Cap
- removed C17: 10u, hellen-one-common:C0603, symbol hellen-one-common:Cap
- removed D10, D11, D12, D13, D14: B5819W, Diode_SMD:D_SOD-123, symbol hellen-one-common:1N4148WS
- removed D4, D6, D7, D8: LED-GREEN-0805, hellen-one-common:LED-0805, symbol hellen-one-common:LED
- removed D5, D9: 1N4148WS, hellen-one-common:SOD-323, symbol hellen-one-common:1N4148WS
- removed G1, G2, G3, G5: PROTO_AREA, hellen-one-common:PROTO_AREA, symbol hellen-one-common:PROTO_AREA
- removed G4: DISCLAIMER, rusefi_lib:Off_Road_Disclaimer, symbol Off_Road_Disclaimer:Disclaimer
- removed G6: LOGO, hellen-one-common:LOGO, symbol hellen-one-common:LOGO
- removed G7: LOGO, rusefi_lib:LOGO, symbol logo:LOGO
- removed J1: USB_B_Mini, hellen-one-common:USB-MINI-B-VERTICAL, symbol hellen-one-common:USB_B_Mini
- removed J10: AudioJack_THR, hellen-one-common:Jack_3.5mm_PJ-3250-5A, symbol hellen-one-common:AudioJack_THR
- removed J2, J3, J4, J5, J6: Conn_01x01, TestPoint:TestPoint_Pad_D2.0mm, symbol Connector_Generic:Conn_01x01
- removed J7: Conn_01x08, Connector_PinHeader_2.54mm:PinHeader_1x08_P2.54mm_Vertical, symbol Connector_Generic:Conn_01x08
- removed J8: Conn_01x06, Connector_PinHeader_2.54mm:PinHeader_1x06_P2.54mm_Vertical, symbol Connector_Generic:Conn_01x06
- removed M1: Module-motor-driver-0.1, hellen-one-motor-driver-0.1:motor-driver, symbol hellen-one-motor-driver-0.1:Module-motor-driver-0.1
- removed M11: Module-vr-discrete-0.4, hellen-one-vr-discrete-0.4:vr-discrete, symbol vr-discrete-0.4:Module-vr-discrete-0.4
- removed M3: mega-mcu144-0.1, hellen-one-mega-mcu144-0.1:mega-mcu144, symbol mega-mcu144-0.1:mega-mcu144-0.1
- removed M5: Module-knock-0.2, hellen-one-knock-0.2:knock, symbol hellen-one-knock-0.2:Module-knock-0.2
- removed M6: Module-output-0.3, hellen-one-output-0.3:output, symbol hellen-one-output-0.3:Module-output-0.3
- removed M7: Module-ign8-0.2, hellen-one-ign8-0.2:ign8, symbol hellen-one-ign8-0.2:Module-ign8-0.2
- removed M8: Module-power_12and5V-0.1, hellen-one-power_12and5V-0.1:power_12and5V, symbol power_12and5V-0.1:Module-power_12and5V-0.1
- removed M9: Module-wbo-0.5, hellen-one-wbo-0.5:wbo, symbol hellen-one-wbo-0.5:Module-wbo-0.5
- removed unit 2 of P1
- removed P10, P11, P12, P13, P14, P15, P16, P17, P2, P20, P28, P3, P4, P40, P41, P43, P44, P45, P46, P48, P49, P5, P56, P6, P61, P63, P64, P66, P67, P68, P69, P7, P74, P8, P80, P9: Pad, hellen-one-common:PAD-TH, symbol hellen-one-common:Pad
- removed R10, R11, R12, R13, R2, R3, R8, R9: Jumper-Pad-Pad, hellen-one-common:PAD-0805-PAD, symbol hellen-one-common:Jumper-Pad-Pad
- removed R16, R17: 5.1k, hellen-one-common:R0603, symbol hellen-one-common:Res
- removed R20: 1.6k, hellen-one-common:R0603, symbol hellen-one-common:Res
- removed R21: 750, hellen-one-common:R0603, symbol hellen-one-common:Res
- removed R23: 0, hellen-one-common:R0603, symbol hellen-one-common:Res
- removed U3: MCP6002-xSN, Package_SO:SOIC-8_3.9x4.9mm_P1.27mm, symbol Amplifier_Operational:MCP6002-xSN
- added D1, D2, D4: B5819W, hellen-one-common:SOD-123, symbol hellen-one-common:1N4148WS
- added D5: SS34, Diode_SMD:D_SMA, symbol Diode:SS34
- added F3: 12H1500D, hellen-one-common:PAD-1206-PAD, symbol hellen-one-common:Fuse-Pad-Pad
- added J1: Conn_01x05_Male, Connector_Molex:Molex_SPOX_5267-05A_1x05_P2.50mm_Vertical, symbol Connector:Conn_01x05_Pin
- added J2: USB_B_Mini, hellen-one-common:USB-MINI-B-VERTICAL, symbol hellen-one-common:USB_B_Mini
- added M1: Module-power_12and5V-0.3, hellen-one-power_12and5V-0.3:power_12and5V, symbol hellen-one-power_12and5V:Module-power_12and5V-0.3
- added M2: Module-knock-0.2, hellen-one-knock-0.2:knock, symbol hellen-one-knock-0.2:Module-knock-0.2
- added M3: Module-vr-discrete-0.5, hellen-one-vr-discrete-0.5:vr-discrete, symbol hellen-one-vr-discrete-0.5:Module-vr-discrete-0.5
- added M4: Module-vr-max9924-0.1, hellen-one-vr-max9924-0.1:vr-max9924, symbol vr-max9924:Module-vr-max9924-0.1
- added M5: Module-motor-driver-0.1, hellen-one-motor-driver-0.1:motor-driver, symbol motor-driver:Module-motor-driver-0.1
- added M6: Module-wbo-0.5, hellen-one-wbo-0.5:wbo, symbol hellen-one-wbo-0.5:Module-wbo-0.5
- added M7: Module:mega-mcu100/0.3, hellen-one-mega-mcu100-0.3:mega-mcu100, symbol hellen-one-mega-mcu100-0.3:Module{colon}mega-mcu100/0.3
- added M8: Module-can-0.1, hellen-one-can-0.1:can, symbol hellen-one-can-0.1:Module-can-0.1
- added P2: 368255-2, footprints:368255-2, symbol 368255-2:368255-2
- added Q1: AO3400A, Package_TO_SOT_SMD:SOT-23, symbol Transistor_FET:AO3400A
- added R1, R13: 4.7k, hellen-one-common:R0603, symbol hellen-one-common:Res
- added R10, R11, R12: 10k, hellen-one-common:R0805, symbol hellen-one-common:Res
- added R14: 1k, hellen-one-common:R0603, symbol hellen-one-common:Res
- added R2: 33k, hellen-one-common:R0603, symbol hellen-one-common:Res
- added R3: 6.8k, hellen-one-common:R0603, symbol hellen-one-common:Res
- added R5, R6: 0, hellen-one-common:R0603, symbol hellen-one-common:Res
- added R7, R8, R9: DNP, hellen-one-common:R0805, symbol hellen-one-common:Res
- added U1: BTS6143D, Package_TO_SOT_SMD:TO-252-4, symbol Power_Management:BTS6143D
- D3: value 1N4148WS -> B5819W; footprint hellen-one-common:SOD-323 -> hellen-one-common:SOD-123; LCSC C2128 -> C8598
- F1: value Fuse-Pad-Pad -> 12H1500D; LCSC (none) -> C182446; MyComment DNP -> (none)
- F2: value Fuse-Pad-Pad -> 12H1500D
- P1: footprint hellen121vag:368255-2 -> footprints:368255-2
- R4: LCSC C17477 -> C17477
Connections:
- net +ETB_OUT is gone; now on net +12V_RAW: P1.117
- net OUT_VVT1_2 is gone; now on net GND: P1.115
- net OUT_VVT2_B2 is gone; now on net +12V: P1.120
- net +12V: now also F2.1, F3.1, P2.23, P2.24, R2.2, U1.3 (Vbb)
- net +12V_RAW: now also D3.1 (K), D1.1 (K), D2.1 (K), D4.1 (K), M1.V3 (V12_RAW); no longer F1.2
- net +5V: now also M1.E4 (V5), M7.N22 (VCC)
- net +5VA: now also M2.E1 (V5A), M3.E4 (V5_IN), M4.E4 (V5_IN), M6.W1 (V5_IN), M7.E1 (V5A_SWITCHABLE), M7.W2 (V5A_SWITCHABLE), M8.V1 (V5), R7.2, R8.2, R9.2
- net +5VP: now also M1.V4 (5VP), P2.106, P2.107, P2.71, P2.72, P2.73, P2.74, P2.75, P2.76, P2.77, P2.78, P2.79, P2.80, R1.1
- net GND: now also P1.114, P1.3, D5.2 (A), J1.4 (Pin_4), J1.5 (Pin_5), J2.5 (GND), J2.6 (Shield), M1.S1 (GND), M2.E2 (GND), M3.G (GND), M4.G (GND), M5.G (GND), M6.E6 (LSU_H-), M6.G (GND), M7.G (GND), M8.E1 (GND), Q1.2 (S), R13.2, R14.2, R3.1; no longer P1.1, P1.2
- net GNDA: now also M7.W1 (GNDA), P2.113, P2.52, P2.53, P2.54, P2.55, P2.56, P2.57, P2.58, P2.59, P2.60, P2.61, P2.62, P2.64, P2.66, P2.68, P2.98, P2.99, R10.1, R11.1, R12.1
- net IGN1: now also M7.W10 (IGN1_(PC13))
- net IGN2: now also M7.W9 (IGN2_(PE5))
- net IGN3: now also M7.W8 (IGN3_(PE4))
- net IGN4: now also M7.W7 (IGN4_(PE3))
- net IGN5: now also M7.W6 (IGN5_(PE2))
- net IGN6: now also M7.W5 (IGN6_(PB8))
- net INJ1: now also M7.E17 (OUT_INJ1_(PD3))
- net INJ2: now also M7.E16 (OUT_INJ2_(PA9))
- net INJ3: now also M7.E15 (OUT_INJ3_(PD11))
- net INJ4: now also M7.E14 (OUT_INJ4_(PD10))
- net INJ5: now also M7.E13 (OUT_INJ5_(PD2))
- net INJ6: now also M7.E12 (OUT_INJ6_(PA8))
- net IN_VIGN: now also F1.2, M1.V2 (IN_VIGN); no longer D3.1 (K)
- net VBAT: now also M1.E1 (VBAT), M7.N17 (VBAT)
- net VBUS: now also J1.1 (Pin_1), J2.1 (VBUS), M7.N1 (VBUS)
- net VIGN: now also M1.E3 (VIGN), M7.E5 (IN_VIGN_(PA5))
- net at R4.1: now also M1.E6 (PG_5VP)
- net +12V_PERM: now reaches P1.116
- net +12V_PERM: now also M1.V1 (V12_PERM)
- net PIN119: now reaches P1.119
- net PIN119: now also M6.E5 (LSU_H+)
- net PIN121: now reaches P1.121
- net PIN121: no longer F2.1
- net PIN108: now reaches F1.1
- net PIN108: now also P2.108; no longer P1.3
- net PIN4: now reaches P1.4
- net PIN16: now reaches D3.2 (A)
- net PIN16: now also P2.16
- net -ETB_OUT renamed PIN118
- net LSU_HEAT- renamed PIN5
- net OUT_TACH renamed PG_5VP
- net PG_5VP: now also M7.N12 (SPI3_MOSI_(PC12))
- new net: F3.2, M5.N2 (12V_IN), M5.S1 (12V_IN)
- new net: M7.N14a (LED_GREEN), Q1.1 (G), R13.1
- new net: Q1.3 (D), U1.2 (IN)
- new net: M6.J1 (SEL1), M6.J_GND1 (PULL_DOWN1)
- new net: R14.1, U1.4 (IS)
- new net +3.3V: M5.W5 (3V3_IN), M7.N21 (V33)
- new net +3.3VA: M7.N15 (V33_SWITCHABLE), M8.V2 (CAN_VIO)
- new net ADC3: M7.S15 (IN_KNOCK_(PA2)), R5.2, R6.2
- new net DC1_DIR: M5.W4 (DIR), M7.E21 (OUT_PWM4_(PC8))
- new net DC1_DIS_W1: M5.W1 (DIS), M7.E8 (SPI2_MISO_(PB14))
- new net DC1_PWM: M5.W2 (PWM), M7.E20 (OUT_PWM3_(PC7))
- new net DC2_DIR: M7.E9 (SPI2_MOSI_(PB15))
- new net DC2_DIS: M7.N4 (USBID_(PA10))
- new net DC2_PWM: M7.E22 (OUT_PWM5_(PC9))
- new net E6INJ7CANRX: M7.E6 (SPI2_CS_/_CAN2_RX_(PB12)), M8.V6 (CAN_RX)
- new net E7INJ8CANTX: M7.E7 (SPI2_SCK_/_CAN2_TX_(PB13)), M8.V5 (CAN_TX)
- new net EGT/SPI_CS: M7.N9 (SPI3_CS_(PA15))
- new net INTERNAL_MAP: M7.S12 (IN_MAP2_(PC1))
- new net IN_AUX3: M7.S7 (IN_AUX3_(PA7))
- new net IN_KNOCK: M2.E3 (OUT_KNOCK), R5.1
- new net IN_VMAIN: M7.S6 (IN_AUX4_(PC5)), R2.1, R3.2
- new net LS1: M7.E11 (OUT_INJ7_(PD15))
- new net LS2: M7.E10 (OUT_INJ8_(PD12))
- new net LS3: M7.E18 (OUT_PWM1_(PD13))
- new net LS4: M7.E19 (OUT_PWM2_(PC6))
- new net LS_HOT1: M7.W4 (IGN7_(PB9))
- new net LS_HOT2: M7.W3 (IGN8_(PE6))
- new net MISO3: M7.N11 (SPI3_MISO_(PC11))
- new net PIN1: M5.S3 (OUT+), P1.1
- new net PIN10: P2.10
- new net PIN100: P2.100
- new net PIN101: P2.101
- new net PIN102: M6.E4 (LSU_Rtrim), P2.102
- new net PIN103: M6.E3 (LSU_Ip), P2.103
- new net PIN104: M6.E2 (LSU_Vm), P2.104
- new net PIN105: M6.E1 (LSU_Un), P2.105
- new net PIN109: P2.109
- new net PIN11: P2.11
- new net PIN110: P2.110
- new net PIN111: P2.111
- new net PIN112: P2.112
- new net PIN12: P2.12
- new net PIN13: P2.13
- new net PIN14: D1.2 (A), P2.14
- new net PIN15: D2.2 (A), P2.15
- new net PIN17: M3.W2 (VR+), P2.17
- new net PIN18: M3.W1 (VR-), P2.18
- new net PIN19: M4.W2 (VR+), P2.19
- new net PIN2: M5.S2 (OUT-), P1.2
- new net PIN20: M4.W1 (VR-), P2.20, R1.2
- new net PIN21: P2.21
- new net PIN22: P2.22
- new net PIN25: P2.25
- new net PIN26: P2.26
- new net PIN27: P2.27
- new net PIN28: P2.28
- new net PIN29: P2.29
- new net PIN30: P2.30
- new net PIN31: P2.31
- new net PIN32: P2.32
- new net PIN33: P2.33
- new net PIN34: M7.S2 (IN_D3_(PE14)), P2.34
- new net PIN35: M7.S3 (IN_D2_(PE13)), P2.35
- new net PIN36: M7.S4 (IN_D1_(PE12)), P2.36
- new net PIN37: M7.S13 (IN_MAP1_(PC0)), P2.37
- new net PIN38: M7.S18 (IN_TPS_(PA4)), P2.38
- new net PIN39: M7.S9 (IN_AUX1_(PB0)), P2.39
- new net PIN40: M7.S11 (IN_O2S_/_CAN_WAKEUP_(PA0)), P2.40
- new net PIN41: M7.S10 (IN_O2S2_(PA1)), P2.41
- new net PIN42: M7.S17 (IN_VSS_(PE11)), P2.42
- new net PIN43: D5.1 (K), P2.43, U1.1 (OUT), U1.5 (OUT)
- new net PIN44: P2.44
- new net PIN45: P2.45
- new net PIN46: P2.46
- new net PIN47: P2.47
- new net PIN48: P2.48
- new net PIN49: P2.49
- new net PIN50: P2.50
- new net PIN51: P2.51
- new net PIN6: M7.N14 (UART2_RX_(PD6)), P2.6
- new net PIN63: M7.S20 (IN_IAT_(PC3)), P2.63
- new net PIN65: M7.S21 (IN_CLT_(PC2)), P2.65
- new net PIN67: P2.67
- new net PIN69: P2.69
- new net PIN7: M7.N13 (UART2_TX_(PD5)), P2.7
- new net PIN70: P2.70
- new net PIN8: P2.8
- new net PIN81: M2.W1 (IN_KNOCK), P2.81
- new net PIN82: M6.W4 (CANH), M7.W11 (CANH), P2.82
- new net PIN83: M6.W3 (CANL), M7.W12 (CANL), P2.83
- new net PIN84: M7.S14 (IN_CRANK_(PB1)), P2.84, R10.2, R7.1
- new net PIN85: M7.S16 (IN_CAM_(PA6)), P2.85, R11.2, R8.1
- new net PIN86: P2.86
- new net PIN87: P2.87
- new net PIN88: D4.2 (A), P2.88
- new net PIN89: M7.S1 (IN_D4_(PE15)), P2.89, R12.2, R9.1
- new net PIN9: P2.9
- new net PIN90: M7.S19 (IN_PPS_(PA3)), P2.90
- new net PIN91: M7.S8 (IN_AUX2_(PC4/PE9)), P2.91
- new net PIN92: P2.92
- new net PIN93: P2.93
- new net PIN94: P2.94
- new net PIN95: P2.95
- new net PIN96: P2.96
- new net PIN97: P2.97
- new net PWR_EN: M1.E5 (EN_5VP), M7.N20 (OUT_PWR_EN_(PE10))
- new net SCK3: M7.N10 (SPI3_SCK_(PC10))
- new net USB+: J1.3 (Pin_3), J2.3 (D+), M7.N3 (USBP_(PA12))
- new net USB-: J1.2 (Pin_2), J2.2 (D-), M7.N2 (USBM_(PA11))
- new net VREF1: M2.W2 (VREF), M7.S22 (VREF1)
- new net VR_DISCRETE: M3.E3 (OUT), M7.N18 (UART8_RX_(PE0))
- new net VR_DISCRETE_A: M3.E2 (OUT_A), R6.1
- new net VR_DISCRETE_THR: M3.E1 (Thresh_IN), M7.E23 (OUT_PWM6_(PD14))
- new net VR_MAX9924: M4.E3 (OUT), M7.N19 (UART8_TX_(PE1))
- no-connect marks 70 -> 22
Other:
- added sheet EGT (egt.kicad_sch)
- added sheet Ignition (IGN6.kicad_sch)
- added sheet Injector (INJ6.kicad_sch)
- added sheet LS (LS4.kicad_sch)
- added sheet LS HOT (LS_HOT.kicad_sch)
- note added: "#0"
- note added: "3.5A MAX Always hot capable"
- note added: "3.5A MAX Solenoid load capable"
- note added: "Configurable "BUTTON" pulls"
- note added: "DC Motor"
- note added: "Flyback diodes"
- note added: "Install a 4.7 kOhm R1 resistor for using VR2- as a hall sensor input"
- note added: "LS & HS outputs"
- note added: "Move the resistor from position R143 to R145 to enable the CAN WAKEUP function. The AUX1 analog input will be unavailable."
- note added: "Move the resistor from position R6 to R5 to use ADC3 for receiving the analog signal VR-DISCRETE instead of the knock signal"
- note added: "Pin 8 may be used for shielding VR signals"
- note added: "Pin Name Recommended function B8 OUT_LS_HOT2 Fan Relay B9 OUT_LS_HOT1 Main Relay B16 OUT_LS4 Fuel Pump Replay B18 OUT_LS2 Idle Air Valve C8 GND VR Shield C15 IN_AUX3 Fuel Pressure D10 IN_BUTTON2 A/C Request All inputs are 12V-tolerant"
- note removed: "#1"
- note removed: "Board info"
- note removed: "ETB driver"
- note removed: "LEDs"
- note removed: "Ouputs"
- note removed: "Power"
- note removed: "Prototype areas"
- note removed: "TODO: knock 2"
- note removed: "http://rusefi.com/s/hellen121vag"
- note removed: "to ETB driver"

Commit message: awsw
Parts:
- M5: value Module-motor-driver-0.1 -> Module-wbo-0.5; footprint hellen-one-motor-driver-0.1:motor-driver -> hellen-one-wbo-0.5:wbo
- M6: value Module-wbo-0.5 -> Module:mega-mcu100/0.3; footprint hellen-one-wbo-0.5:wbo -> hellen-one-mega-mcu100-0.3:mega-mcu100; FITTED (none) -> False; PUBLISHER (none) -> qwerty-off; SUPPLIER 1 (none) -> Mouser; SUPPLIER 2 (none) -> Digi-Key; SUPPLIER 3 (none) -> LCSC; SUPPLIER PART NUMBER 1 (none) -> *; SUPPLIER PART NUMBER 2 (none) -> *; TYPE (none) -> Module
- M7: value Module:mega-mcu100/0.3 -> Module-can-0.1; footprint hellen-one-mega-mcu100-0.3:mega-mcu100 -> hellen-one-can-0.1:can; FITTED False -> (none); PUBLISHER qwerty-off -> (none); SUPPLIER 1 Mouser -> (none); SUPPLIER 2 Digi-Key -> (none); SUPPLIER PART NUMBER 1 * -> (none); SUPPLIER PART NUMBER 2 * -> (none); TYPE Module -> (none)
- M8: value Module-can-0.1 -> Module-motor-driver-0.1; footprint hellen-one-can-0.1:can -> hellen-one-motor-driver-0.1:motor-driver
- Q1: value AO3400A -> ISL9V3040D3ST; footprint Package_TO_SOT_SMD:SOT-23 -> Package_TO_SOT_SMD:TO-252-2; MyComment (none) -> DNP
- R13: LCSC C21189 -> C23162
- R14: value 1k -> 4.7k; LCSC C21189 -> C23162
Connections:
- net DC1_DIR is gone; now on net PIN82: M5.W4 (DIR), M7.E21 (OUT_PWM4_(PC8))
- net INJ1 is gone; now on net E7INJ8CANTX: M7.E17 (OUT_INJ1_(PD3))
- net INJ3 is gone; now on net INJ2: M7.E15 (OUT_INJ3_(PD11))
- net INJ4 is gone; now on net INJ2: M7.E14 (OUT_INJ4_(PD10))
- net INJ5 is gone; now on net INJ2: M7.E13 (OUT_INJ5_(PD2))
- net LS1 is gone; now on net E6INJ7CANRX: M7.E11 (OUT_INJ7_(PD15))
- net LS2 is gone; now on net E7INJ8CANTX: M7.E10 (OUT_INJ8_(PD12))
- net LS3 is gone; now on net E7INJ8CANTX: M7.E18 (OUT_PWM1_(PD13))
- net LS4 is gone; now on net E6INJ7CANRX: M7.E19 (OUT_PWM2_(PC6))
- net LS_HOT2 is gone; now on net LS_HOT1: M7.W3 (IGN8_(PE6))
- net +5VA: now also M5.W1 (DIS), M6.E1 (LSU_Un), M6.W2 (CAN_VIO)
- net DC1_DIS_W1: no longer M5.W1 (DIS)
- net GND: now also Q1.3 (D), U1.2 (IN)
- net IGN2: now also M6.W9 (VDDA)
- net IGN3: now also M6.W8 (V33_OUT)
- net IGN4: now also M6.W7 (SWCLK)
- net IGN5: now also M6.W6 (SWDIO)
- net IGN6: now also M6.W5 (nReset)
- net LS_HOT1: now also M6.W3 (CANL), M6.W4 (CANH), M7.N14a (LED_GREEN), Q1.1 (G), R13.1, R14.1, U1.4 (IS)
- net PIN105: no longer M6.E1 (LSU_Un)
- net PIN119: no longer M6.E5 (LSU_H+)
- net PIN2: now also M8.S2 (CANH)
- net PIN82: no longer M6.W4 (CANH)
- net PIN83: now also M5.W3 (SCLK); no longer M6.W3 (CANL)
- net VIGN: now also M6.E5 (LSU_H+)
- net Net-(F3-Pad2): now reaches M8.S1 (CANL)

Commit message: wwew
Parts:
- removed J1: Conn_01x05_Male, Connector_Molex:Molex_SPOX_5267-05A_1x05_P2.50mm_Vertical, symbol Connector:Conn_01x05_Pin
- removed J2: USB_B_Mini, hellen-one-common:USB-MINI-B-VERTICAL, symbol hellen-one-common:USB_B_Mini
- removed M5: Module-wbo-0.5, hellen-one-wbo-0.5:wbo, symbol motor-driver:Module-motor-driver-0.1
- removed M6: Module:mega-mcu100/0.3, hellen-one-mega-mcu100-0.3:mega-mcu100, symbol hellen-one-wbo-0.5:Module-wbo-0.5
- removed M7: Module-can-0.1, hellen-one-can-0.1:can, symbol hellen-one-mega-mcu100-0.3:Module{colon}mega-mcu100/0.3
- removed M8: Module-motor-driver-0.1, hellen-one-motor-driver-0.1:motor-driver, symbol hellen-one-can-0.1:Module-can-0.1
- removed P2: 368255-2, footprints:368255-2, symbol 368255-2:368255-2
- removed Q1: ISL9V3040D3ST, Package_TO_SOT_SMD:TO-252-2, symbol Transistor_FET:AO3400A
- removed R13, R14: 4.7k, hellen-one-common:R0603, symbol hellen-one-common:Res
- removed U1: BTS6143D, Package_TO_SOT_SMD:TO-252-4, symbol Power_Management:BTS6143D
- added J21: Conn_01x05_Male, Connector_Molex:Molex_SPOX_5267-05A_1x05_P2.50mm_Vertical, symbol Connector:Conn_01x05_Pin
- added J22: USB_B_Mini, hellen-one-common:USB-MINI-B-VERTICAL, symbol hellen-one-common:USB_B_Mini
- added M5: Module-wbo-0.5, hellen-one-wbo-0.5:wbo, symbol hellen-one-wbo-0.5:Module-wbo-0.5
- added M6: Module:mega-mcu100/0.3, hellen-one-mega-mcu100-0.3:mega-mcu100, symbol hellen-one-mega-mcu100-0.3:Module{colon}mega-mcu100/0.3
- added M7: Module-can-0.1, hellen-one-can-0.1:can, symbol hellen-one-can-0.1:Module-can-0.1
- added M8: Module-motor-driver-0.1, hellen-one-motor-driver-0.1:motor-driver, symbol motor-driver:Module-motor-driver-0.1
- added unit 2 of P1
- added Q7: AO3400A, Package_TO_SOT_SMD:SOT-23, symbol Transistor_FET:AO3400A
- added R15: 4.7k, hellen-one-common:R0603, symbol hellen-one-common:Res
- added R54: 1k, hellen-one-common:R0603, symbol hellen-one-common:Res
- added U10: BTS6143D, Package_TO_SOT_SMD:TO-252-4, symbol Power_Management:BTS6143D
- P1: footprint footprints:368255-2 -> 368255-2:368255-2
Connections:
- net +12V: now also P1.23, P1.24, U10.3 (Vbb)
- net +3.3V: now also M6.N21 (V33), M8.W5 (3V3_IN)
- net +3.3VA: now also M6.N15 (V33_SWITCHABLE), M7.V2 (CAN_VIO)
- net +5V: now also M6.N22 (VCC)
- net +5VA: now also M5.W1 (V5_IN), M6.E1 (V5A_SWITCHABLE), M6.W2 (V5A_SWITCHABLE), M7.V1 (V5)
- net +5VP: now also P1.106, P1.107, P1.71, P1.72, P1.73, P1.74, P1.75, P1.76, P1.77, P1.78, P1.79, P1.80
- net ADC3: now also M6.S15 (IN_KNOCK_(PA2))
- net DC1_DIS_W1: now also M6.E8 (SPI2_MISO_(PB14)), M8.W1 (DIS)
- net DC1_PWM: now also M6.E20 (OUT_PWM3_(PC7)), M8.W2 (PWM)
- net DC2_DIR: now also M6.E9 (SPI2_MOSI_(PB15))
- net DC2_DIS: now also M6.N4 (USBID_(PA10))
- net DC2_PWM: now also M6.E22 (OUT_PWM5_(PC9))
- net E6INJ7CANRX: now also M6.E6 (SPI2_CS_/_CAN2_RX_(PB12)), M7.V6 (CAN_RX)
- net E7INJ8CANTX: now also M6.E7 (SPI2_SCK_/_CAN2_TX_(PB13)), M7.V5 (CAN_TX)
- net EGT/SPI_CS: now also M6.N9 (SPI3_CS_(PA15))
- net GND: now also J21.4 (Pin_4), J21.5 (Pin_5), J22.5 (GND), J22.6 (Shield), M5.E6 (LSU_H-), M5.G (GND), M6.G (GND), M7.E1 (GND), M8.G (GND), Q7.2 (S), R15.2, R54.2
- net GNDA: now also M6.W1 (GNDA), P1.113, P1.52, P1.53, P1.54, P1.55, P1.56, P1.57, P1.58, P1.59, P1.60, P1.61, P1.62, P1.64, P1.66, P1.68, P1.98, P1.99
- net IGN1: now also M6.W10 (IGN1_(PC13))
- net IGN2: now also M6.W9 (IGN2_(PE5))
- net IGN3: now also M6.W8 (IGN3_(PE4))
- net IGN4: now also M6.W7 (IGN4_(PE3))
- net IGN5: now also M6.W6 (IGN5_(PE2))
- net IGN6: now also M6.W5 (IGN6_(PB8))
- net INJ2: now also M6.E16 (OUT_INJ2_(PA9))
- net INJ6: now also M6.E12 (OUT_INJ6_(PA8))
- net INTERNAL_MAP: now also M6.S12 (IN_MAP2_(PC1))
- net IN_AUX3: now also M6.S7 (IN_AUX3_(PA7))
- net IN_VMAIN: now also M6.S6 (IN_AUX4_(PC5))
- net LS_HOT1: now also M6.W4 (IGN7_(PB9))
- net MISO3: now also M6.N11 (SPI3_MISO_(PC11))
- net PG_5VP: now also M6.N12 (SPI3_MOSI_(PC12))
- net PIN1: now also M8.S3 (OUT+)
- net PIN10: now also P1.10
- net PIN100: now also P1.100
- net PIN101: now also P1.101
- net PIN102: now also M5.E4 (LSU_Rtrim), P1.102
- net PIN103: now also M5.E3 (LSU_Ip), P1.103
- net PIN104: now also M5.E2 (LSU_Vm), P1.104
- net PIN105: now also M5.E1 (LSU_Un), P1.105
- net PIN108: now also P1.108
- net PIN109: now also P1.109
- net PIN11: now also P1.11
- net PIN110: now also P1.110
- net PIN111: now also P1.111
- net PIN112: now also P1.112
- net PIN119: now also M5.E5 (LSU_H+)
- net PIN12: now also P1.12
- net PIN13: now also P1.13
- net PIN14: now also P1.14
- net PIN15: now also P1.15
- net PIN16: now also P1.16
- net PIN17: now also P1.17
- net PIN18: now also P1.18
- net PIN19: now also P1.19
- net PIN2: now also M8.S2 (OUT-)
- net PIN20: now also P1.20
- net PIN21: now also P1.21
- net PIN22: now also P1.22
- net PIN25: now also P1.25
- net PIN26: now also P1.26
- net PIN27: now also P1.27
- net PIN28: now also P1.28
- net PIN29: now also P1.29
- net PIN30: now also P1.30
- net PIN31: now also P1.31
- net PIN32: now also P1.32
- net PIN33: now also P1.33
- net PIN34: now also M6.S2 (IN_D3_(PE14)), P1.34
- net PIN35: now also M6.S3 (IN_D2_(PE13)), P1.35
- net PIN36: now also M6.S4 (IN_D1_(PE12)), P1.36
- net PIN37: now also M6.S13 (IN_MAP1_(PC0)), P1.37
- net PIN38: now also M6.S18 (IN_TPS_(PA4)), P1.38
- net PIN39: now also M6.S9 (IN_AUX1_(PB0)), P1.39
- net PIN40: now also M6.S11 (IN_O2S_/_CAN_WAKEUP_(PA0)), P1.40
- net PIN41: now also M6.S10 (IN_O2S2_(PA1)), P1.41
- net PIN42: now also M6.S17 (IN_VSS_(PE11)), P1.42
- net PIN43: now also P1.43, U10.1 (OUT), U10.5 (OUT)
- net PIN44: now also P1.44
- net PIN45: now also P1.45
- net PIN46: now also P1.46
- net PIN47: now also P1.47
- net PIN48: now also P1.48
- net PIN49: now also P1.49
- net PIN50: now also P1.50
- net PIN51: now also P1.51
- net PIN6: now also M6.N14 (UART2_RX_(PD6)), P1.6
- net PIN63: now also M6.S20 (IN_IAT_(PC3)), P1.63
- net PIN65: now also M6.S21 (IN_CLT_(PC2)), P1.65
- net PIN67: now also P1.67
- net PIN69: now also P1.69
- net PIN7: now also M6.N13 (UART2_TX_(PD5)), P1.7
- net PIN70: now also P1.70
- net PIN8: now also P1.8
- net PIN81: now also P1.81
- net PIN82: now also M5.W4 (CANH), M6.W11 (CANH), P1.82
- net PIN83: now also M5.W3 (CANL), M6.W12 (CANL), P1.83
- net PIN84: now also M6.S14 (IN_CRANK_(PB1)), P1.84
- net PIN85: now also M6.S16 (IN_CAM_(PA6)), P1.85
- net PIN86: now also P1.86
- net PIN87: now also P1.87
- net PIN88: now also P1.88
- net PIN89: now also M6.S1 (IN_D4_(PE15)), P1.89
- net PIN9: now also P1.9
- net PIN90: now also M6.S19 (IN_PPS_(PA3)), P1.90
- net PIN91: now also M6.S8 (IN_AUX2_(PC4/PE9)), P1.91
- net PIN92: now also P1.92
- net PIN93: now also P1.93
- net PIN94: now also P1.94
- net PIN95: now also P1.95
- net PIN96: now also P1.96
- net PIN97: now also P1.97
- net PWR_EN: now also M6.N20 (OUT_PWR_EN_(PE10))
- net SCK3: now also M6.N10 (SPI3_SCK_(PC10))
- net USB+: now also J21.3 (Pin_3), J22.3 (D+), M6.N3 (USBP_(PA12))
- net USB-: now also J21.2 (Pin_2), J22.2 (D-), M6.N2 (USBM_(PA11))
- net VBAT: now also M6.N17 (VBAT)
- net VBUS: now also J21.1 (Pin_1), J22.1 (VBUS), M6.N1 (VBUS)
- net VIGN: now also M6.E5 (IN_VIGN_(PA5))
- net VREF1: now also M6.S22 (VREF1)
- net VR_DISCRETE: now also M6.N18 (UART8_RX_(PE0))
- net VR_DISCRETE_THR: now also M6.E23 (OUT_PWM6_(PD14))
- net VR_MAX9924: now also M6.N19 (UART8_TX_(PE1))
- net at F3.2: now also M8.N2 (12V_IN), M8.S1 (12V_IN)
- new net: M6.N14a (LED_GREEN), Q7.1 (G), R15.1
- new net: Q7.3 (D), U10.2 (IN)
- new net: R54.1, U10.4 (IS)
- new net: M5.J1 (SEL1), M5.J_GND1 (PULL_DOWN1)
- new net DC1_DIR: M6.E21 (OUT_PWM4_(PC8)), M8.W4 (DIR)
- new net INJ1: M6.E17 (OUT_INJ1_(PD3))
- new net INJ3: M6.E15 (OUT_INJ3_(PD11))
- new net INJ4: M6.E14 (OUT_INJ4_(PD10))
- new net INJ5: M6.E13 (OUT_INJ5_(PD2))
- new net LS1: M6.E11 (OUT_INJ7_(PD15))
- new net LS2: M6.E10 (OUT_INJ8_(PD12))
- new net LS3: M6.E18 (OUT_PWM1_(PD13))
- new net LS4: M6.E19 (OUT_PWM2_(PC6))
- new net LS_HOT2: M6.W3 (IGN8_(PE6))
Other:
- company: andreika @ rusEFI.com -> andreika @ rusEFI.comm
