File: IGN6.kicad_sch (KiCad schematic)
At the start: 24 parts, among them Q2 ISL9V3040D3ST, Q3 ISL9V3040D3ST, Q4 ISL9V3040D3ST, Q5 ISL9V3040D3ST, Q6 ISL9V3040D3ST, Q7 ISL9V3040D3ST

Commit message: wq
Parts:
- renumbered F9 to F10, F4 to F5, F5 to F6, F6 to F7, F7 to F8, F8 to F9
Changed lines of the file:
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@@
 		(on_board yes)
 		(dnp no)
-		(property "Reference" "F5"
+		(property "Reference" "F6"
 			(at 114.3 81.28 90)
 			(effects
@@
 			(project "hellen121vag"
 				(path "/45c1f041-3b7c-4036-abe9-e26621c05a73/25e70622-4c27-4350-9ebe-0dc5c0c1dcd9"
-					(reference "F5")
+					(reference "F6")
 					(unit 1)
 				)
@@
 		(on_board yes)
 		(dnp no)
-		(property "Reference" "F9"
+		(property "Reference" "F10"
 			(at 161.29 109.22 90)
 			(effects
@@
 			(project "hellen121vag"
 				(path "/45c1f041-3b7c-4036-abe9-e26621c05a73/25e70622-4c27-4350-9ebe-0dc5c0c1dcd9"
-					(reference "F9")
+					(reference "F10")
 					(unit 1)
 				)
@@
 		(on_board yes)
 		(dnp no)
-		(property "Reference" "F8"
+		(property "Reference" "F9"
 			(at 161.29 81.28 90)
 			(effects
@@
 			(project "hellen121vag"
 				(path "/45c1f041-3b7c-4036-abe9-e26621c05a73/25e70622-4c27-4350-9ebe-0dc5c0c1dcd9"
-					(reference "F8")
+					(reference "F9")
 					(unit 1)
 				)
@@
 		(on_board yes)
 		(dnp no)
-		(property "Reference" "F4"
+		(property "Reference" "F5"
 			(at 114.3 53.34 90)
 			(effects
@@
 			(project "hellen121vag"
 				(path "/45c1f041-3b7c-4036-abe9-e26621c05a73/25e70622-4c27-4350-9ebe-0dc5c0c1dcd9"
-					(reference "F4")
+					(reference "F5")
 					(unit 1)
 				)
@@
 		(on_board yes)
 		(dnp no)
-		(property "Reference" "F6"
+		(property "Reference" "F7"
 			(at 114.3 109.22 90)
 			(effects
@@
 			(project "hellen121vag"
 				(path "/45c1f041-3b7c-4036-abe9-e26621c05a73/25e70622-4c27-4350-9ebe-0dc5c0c1dcd9"
-					(reference "F6")
+					(reference "F7")
 					(unit 1)
 				)
@@
 		(on_board yes)
 		(dnp no)
-		(property "Reference" "F7"
+		(property "Reference" "F8"
 			(at 161.29 53.34 90)
 			(effects
@@
 			(project "hellen121vag"
 				(path "/45c1f041-3b7c-4036-abe9-e26621c05a73/25e70622-4c27-4350-9ebe-0dc5c0c1dcd9"
-					(reference "F7")
-					(unit 1)
-				)
+					(reference "F8")
+					(unit 1)
+				)

Commit message: awsw
Parts:
- Q7: value ISL9V3040D3ST -> AO3400A; footprint Package_TO_SOT_SMD:TO-252-2 -> Package_TO_SOT_SMD:SOT-23; MyComment DNP -> (none)
- R20, R21, R26, R27: value 22 -> 0; footprint hellen-one-common:R0603 -> Resistor_SMD:R_2512_6332Metric; LCSC C23345 -> C25469
- R23, R24: value 0 -> 22; footprint Resistor_SMD:R_2512_6332Metric -> hellen-one-common:R0603; LCSC C25469 -> C23345
- R29, R30: value 0 -> 4.7k; footprint Resistor_SMD:R_2512_6332Metric -> hellen-one-common:R0603; LCSC C25469 -> C23162
Changed lines of the file:
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@@
 			)
 		)
-		(property "Value" "ISL9V3040D3ST"
+		(property "Value" "AO3400A"
 			(at 137.3886 112.903 0)
 			(effects
@@
 			)
 		)
-		(property "Footprint" "Package_TO_SOT_SMD:TO-252-2"
+		(property "Footprint" "Package_TO_SOT_SMD:SOT-23"
 			(at 137.16 109.22 0)
 			(effects
@@
 			)
 		)
-		(property "Datasheet" "~"
+		(property "Datasheet" "http://www.aosmd.com/pdfs/datasheet/AO3400A.pdf"
 			(at 142.24 111.76 0)
 			(effects
@@
 			)
 		)
-		(property "Description" ""
+		(property "Description" "30V Vds, 5.7A Id, N-Channel MOSFET, SOT-23"
 			(at 142.24 111.76 0)
 			(effects
@@
 				)
 				(hide yes)
-			)
-		)
-		(property "LCSC" ""
-			(at 142.24 111.76 0)
-			(effects
-				(font
-					(size 1.27 1.27)
-				)
-				(hide yes)
-			)
-		)
-		(property "MyComment" "DNP"
-			(at 143.764 117.856 0)
-			(effects
-				(font
-					(size 1.27 1.27)
-				)
 			)
 		)
@@
 			)
 		)
-		(property "Value" "0"
+		(property "Value" "4.7k"
 			(at 152.4 78.74 0)
 			(effects
@@
 			)
 		)
-		(property "Footprint" "Resistor_SMD:R_2512_6332Metric"
+		(property "Footprint" "hellen-one-common:R0603"
 			(at 153.67 82.55 0)
 			(effects
@@
 			)
 		)
-		(property "LCSC" "C25469"
+		(property "LCSC" "C23162"
 			(at 157.48 78.74 0)
 			(effects
@@
 			)
 		)
-		(property "Value" "0"
+		(property "Value" "22"
 			(at 105.41 78.74 0)
 			(effects
@@
 			)
 		)
-		(property "Footprint" "Resistor_SMD:R_2512_6332Metric"
+		(property "Footprint" "hellen-one-common:R0603"
 			(at 106.68 82.55 0)
 			(effects
@@
 			)
 		)
-		(property "LCSC" "C25469"
+		(property "LCSC" "C23345"
 			(at 110.49 78.74 0)
 			(effects
@@
 			)
 		)
-		(property "Value" "22"
+		(property "Value" "0"
 			(at 152.4 111.76 0)
 			(effects
@@
 			)
 		)
-		(property "Footprint" "hellen-one-common:R0603"
+		(property "Footprint" "Resistor_SMD:R_2512_6332Metric"
 			(at 151.13 107.95 0)
 			(effects
@@
 			)
 		)
-		(property "LCSC" "C23345"
+		(property "LCSC" "C25469"
 			(at 147.32 111.76 0)
 			(effects
@@
 			)
 		)
-		(property "Value" "0"
+		(property "Value" "22"
 			(at 105.41 106.68 0)
 			(effects
@@
 			)
 		)
-		(property "Footprint" "Resistor_SMD:R_2512_6332Metric"
+		(property "Footprint" "hellen-one-common:R0603"
 			(at 106.68 110.49 0)
 			(effects
@@
 			)
 		)
-		(property "LCSC" "C25469"
+		(property "LCSC" "C23345"
 			(at 110.49 106.68 0)
 			(effects
@@
 			)
 		)
-		(property "Value" "22"
+		(property "Value" "0"
 			(at 152.4 83.82 0)
 			(effects
@@
 			)
 		)
-		(property "Footprint" "hellen-one-common:R0603"
+		(property "Footprint" "Resistor_SMD:R_2512_6332Metric"
 			(at 151.13 80.01 0)
 			(effects
@@
 			)
 		)
-		(property "LCSC" "C23345"
+		(property "LCSC" "C25469"
 			(at 147.32 83.82 0)
 			(effects
@@
 			)
 		)
-		(property "Value" "22"
+		(property "Value" "0"
 			(at 105.41 83.82 0)
 			(effects
@@
 			)
 		)
-		(property "Footprint" "hellen-one-common:R0603"
+		(property "Footprint" "Resistor_SMD:R_2512_6332Metric"
 			(at 104.14 80.01 0)
 			(effects
@@
 			)
 		)
-		(property "LCSC" "C23345"
+		(property "LCSC" "C25469"
 			(at 100.33 83.82 0)
 			(effects
@@
 			)
 		)
-		(property "Value" "0"
+		(property "Value" "4.7k"
 			(at 152.4 106.68 0)
 			(effects
@@
 			)
 		)
-		(property "Footprint" "Resistor_SMD:R_2512_6332Metric"
+		(property "Footprint" "hellen-one-common:R0603"
 			(at 153.67 110.49 0)
 			(effects
@@
 			)
 		)
-		(property "LCSC" "C25469"
+		(property "LCSC" "C23162"
 			(at 157.48 106.68 0)
 			(effects
@@
 			)
 		)
-		(property "Value" "22"
+		(property "Value" "0"
 			(at 105.41 111.76 0)
 			(effects
@@
 			)
 		)
-		(property "Footprint" "hellen-one-common:R0603"
+		(property "Footprint" "Resistor_SMD:R_2512_6332Metric"
 			(at 104.14 107.95 0)
 			(effects
@@
 			)
 		)
-		(property "LCSC" "C23345"
+		(property "LCSC" "C25469"
 			(at 100.33 111.76 0)
 			(effects

Commit message: wwew
Parts:
- renumbered F5 to F4, F6 to F5, F7 to F6, F8 to F7, F9 to F8, F10 to F9, Q2 to Q1, Q3 to Q2, Q4 to Q3, Q5 to Q4, Q6 to Q5, Q7 to Q6, R19 to R18, R20 to R19, R21 to R20, R22 to R21, R23 to R22, R24 to R23, R25 to R24, R26 to R25, R27 to R26, R28 to R27, R29 to R28, R30 to R29

Commit message: wwew
Parts:
- renumbered F9 to F10, F4 to F5, F5 to F6, F6 to F7, F7 to F8, F8 to F9
Changed lines of the file:
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@@
 		(on_board yes)
 		(dnp no)
-		(property "Reference" "F5"
+		(property "Reference" "F6"
 			(at 114.3 81.28 90)
 			(effects
@@
 			(project "hellen121vag"
 				(path "/45c1f041-3b7c-4036-abe9-e26621c05a73/f08b5b09-fcb6-4f5b-8ff2-a721d01c34bf"
-					(reference "F5")
+					(reference "F6")
 					(unit 1)
 				)
@@
 		(on_board yes)
 		(dnp no)
-		(property "Reference" "F9"
+		(property "Reference" "F10"
 			(at 161.29 109.22 90)
 			(effects
@@
 			(project "hellen121vag"
 				(path "/45c1f041-3b7c-4036-abe9-e26621c05a73/f08b5b09-fcb6-4f5b-8ff2-a721d01c34bf"
-					(reference "F9")
+					(reference "F10")
 					(unit 1)
 				)
@@
 		(on_board yes)
 		(dnp no)
-		(property "Reference" "F8"
+		(property "Reference" "F9"
 			(at 161.29 81.28 90)
 			(effects
@@
 			(project "hellen121vag"
 				(path "/45c1f041-3b7c-4036-abe9-e26621c05a73/f08b5b09-fcb6-4f5b-8ff2-a721d01c34bf"
-					(reference "F8")
+					(reference "F9")
 					(unit 1)
 				)
@@
 		(on_board yes)
 		(dnp no)
-		(property "Reference" "F4"
+		(property "Reference" "F5"
 			(at 114.3 53.34 90)
 			(effects
@@
 			(project "hellen121vag"
 				(path "/45c1f041-3b7c-4036-abe9-e26621c05a73/f08b5b09-fcb6-4f5b-8ff2-a721d01c34bf"
-					(reference "F4")
+					(reference "F5")
 					(unit 1)
 				)
@@
 		(on_board yes)
 		(dnp no)
-		(property "Reference" "F6"
+		(property "Reference" "F7"
 			(at 114.3 109.22 90)
 			(effects
@@
 			(project "hellen121vag"
 				(path "/45c1f041-3b7c-4036-abe9-e26621c05a73/f08b5b09-fcb6-4f5b-8ff2-a721d01c34bf"
-					(reference "F6")
+					(reference "F7")
 					(unit 1)
 				)
@@
 		(on_board yes)
 		(dnp no)
-		(property "Reference" "F7"
+		(property "Reference" "F8"
 			(at 161.29 53.34 90)
 			(effects
@@
 			(project "hellen121vag"
 				(path "/45c1f041-3b7c-4036-abe9-e26621c05a73/f08b5b09-fcb6-4f5b-8ff2-a721d01c34bf"
-					(reference "F7")
-					(unit 1)
-				)
+					(reference "F8")
+					(unit 1)
+				)
